File: pcb/plant_sensor-ble.sch (KiCad schematic (older format))
At the start: 3 parts, among them IC1 SPBTLE-RF0

Commit message: Added UART and further work on schematics
Parts:
- C5: footprint (none) -> Capacitors_SMD:C_0805_HandSoldering
- IC1: footprint RF_Module:ST_SPBTLE -> RF_Modules:ST_SPBTLE
- R1: footprint (none) -> Resistors_SMD:R_0805_HandSoldering
Changed lines of the file:
@@
 EESchema Schematic File Version 4
+LIBS:plant_sensor-cache
 EELAYER 26 0
 EELAYER END
@@
 F 0 "IC1" H 4750 3750 50  0000 C CNN
 F 1 "SPBTLE-RF0" H 4950 3650 50  0000 C CNN
-F 2 "RF_Module:ST_SPBTLE" H 5850 2650 50  0001 C CNN
+F 2 "RF_Modules:ST_SPBTLE" H 5850 2650 50  0001 C CNN
 F 3 "http://www.st.com/resource/en/datasheet/spbtle-rf0.pdf" H 4800 3600 50  0001 C CNN
 	1    5350 3200
@@
 F 0 "R1" H 6270 3746 50  0000 L CNN
 F 1 "47K" H 6270 3655 50  0000 L CNN
-F 2 "" V 6130 3700 50  0001 C CNN
+F 2 "Resistors_SMD:R_0805_HandSoldering" V 6130 3700 50  0001 C CNN
 F 3 "~" H 6200 3700 50  0001 C CNN
 	1    6200 3700
@@
 F 0 "C5" V 5802 2650 50  0000 C CNN
 F 1 "1uF" V 5711 2650 50  0000 C CNN
-F 2 "" H 5588 2500 50  0001 C CNN
+F 2 "Capacitors_SMD:C_0805_HandSoldering" H 5588 2500 50  0001 C CNN
 F 3 "~" H 5550 2650 50  0001 C CNN
 	1    5550 2650

Commit message: Smaller MCU updated schematics
Parts:
- renumbered C5 to C2
Connections:
- net labels added: BLE_nRESET
- net labels removed: SPI_BLE_nRESET
Changed lines of the file:
@@
 $Descr A4 11693 8268
 encoding utf-8
-Sheet 2 2
+Sheet 2 3
 Title "BLE"
-Date "2019-02-20"
+Date "2019-02-22"
 Rev ""
 Comp "HuizePD"
@@
 AR Path="/5C6DADA9/5C6DAF3E" Ref="IC1"  Part="1"
 F 0 "IC1" H 4750 3750 50  0000 C CNN
-F 1 "SPBTLE-RF0" H 4950 3650 50  0000 C CNN
+F 1 "SPBTLE-RF0" H 4900 3650 50  0000 C CNN
 F 2 "RF_Modules:ST_SPBTLE" H 5850 2650 50  0001 C CNN
 F 3 "http://www.st.com/resource/en/datasheet/spbtle-rf0.pdf" H 4800 3600 50  0001 C CNN
@@
 P 6200 3900
 AR Path="/5C6DAF4F" Ref="#PWR?"  Part="1"
-AR Path="/5C6DADA9/5C6DAF4F" Ref="#PWR0105"  Part="1"
-F 0 "#PWR0105" H 6200 3650 50  0001 C CNN
+AR Path="/5C6DADA9/5C6DAF4F" Ref="#PWR011"  Part="1"
+F 0 "#PWR011" H 6200 3650 50  0001 C CNN
 F 1 "GND" H 6205 3727 50  0000 C CNN
 F 2 "" H 6200 3900 50  0001 C CNN
@@
 P 5350 3850
 AR Path="/5C6DAF58" Ref="#PWR?"  Part="1"
-AR Path="/5C6DADA9/5C6DAF58" Ref="#PWR0106"  Part="1"
-F 0 "#PWR0106" H 5350 3600 50  0001 C CNN
+AR Path="/5C6DADA9/5C6DAF58" Ref="#PWR09"  Part="1"
+F 0 "#PWR09" H 5350 3600 50  0001 C CNN
 F 1 "GND" H 5355 3677 50  0000 C CNN
 F 2 "" H 5350 3850 50  0001 C CNN
@@
 P 5350 2600
 AR Path="/5C6DAF5F" Ref="#PWR?"  Part="1"
-AR Path="/5C6DADA9/5C6DAF5F" Ref="#PWR0107"  Part="1"
-F 0 "#PWR0107" H 5350 2450 50  0001 C CNN
+AR Path="/5C6DADA9/5C6DAF5F" Ref="#PWR08"  Part="1"
+F 0 "#PWR08" H 5350 2450 50  0001 C CNN
 F 1 "+3V3" H 5365 2773 50  0000 C CNN
 F 2 "" H 5350 2600 50  0001 C CNN
@@
 P 5550 2650
 AR Path="/5C6DAF66" Ref="C?"  Part="1"
-AR Path="/5C6DADA9/5C6DAF66" Ref="C5"  Part="1"
-F 0 "C5" V 5802 2650 50  0000 C CNN
+AR Path="/5C6DADA9/5C6DAF66" Ref="C2"  Part="1"
+F 0 "C2" V 5802 2650 50  0000 C CNN
 F 1 "1uF" V 5711 2650 50  0000 C CNN
 F 2 "Capacitors_SMD:C_0805_HandSoldering" H 5588 2500 50  0001 C CNN
@@
 P 5750 2700
 AR Path="/5C6DAF6D" Ref="#PWR?"  Part="1"
-AR Path="/5C6DADA9/5C6DAF6D" Ref="#PWR0108"  Part="1"
-F 0 "#PWR0108" H 5750 2450 50  0001 C CNN
+AR Path="/5C6DADA9/5C6DAF6D" Ref="#PWR010"  Part="1"
+F 0 "#PWR010" H 5750 2450 50  0001 C CNN
 F 1 "GND" H 5755 2527 50  0000 C CNN
 F 2 "" H 5750 2700 50  0001 C CNN
@@
 	6200 3000 6400 3000
 Text HLabel 4350 3000 0    50   Input ~ 0
-SPI_BLE_nRESET
+BLE_nRESET
 Text HLabel 6400 3500 2    50   Input ~ 0
 BLE_nCS
@@
 Text HLabel 6400 3200 2    50   Input ~ 0
 SPI_CLK
-Text HLabel 6400 3000 2    50   Input ~ 0
+Text HLabel 6400 3000 2    50   Output ~ 0
 BLE_IRQ
 $EndSCHEMATC
