File: pcb/plant_sensor.sch (KiCad schematic (older format))
At the start: 10 parts, among them SW1 SW_Push, U1 STM32L053C8Tx, Y1 8MHz, Y2 32.768kHz

Commit message: Added UART and further work on schematics
Parts:
- added BT1: CR2032, Connectors:CR2032H, symbol Device:Battery_Cell
- added C10: 1uF X5R, Capacitors_SMD:C_0805_HandSoldering, symbol Device:C
- added C11, C7, C8, C9: 100nF, Capacitors_SMD:C_0805_HandSoldering, symbol Device:C
- added D1: RED, LEDs:LED_0805_HandSoldering, symbol Device:LED
- added J1: Conn_ARM_JTAG_SWD_10, Pin_Headers:Pin_Header_Straight_2x05_Pitch1.27mm_SMD, symbol Connector:Conn_ARM_JTAG_SWD_10
- added R3: 10K, Resistors_SMD:R_0805_HandSoldering, symbol Device:R
- added R4: 1K, Resistors_SMD:R_0805_HandSoldering, symbol Device:R
- added R5: FBead, Resistors_SMD:R_0805_HandSoldering, symbol Device:R
- added U2: M95256-WMN6P, Housings_SOIC:SOIC-8_3.9x4.9mm_Pitch1.27mm, symbol Memory_EEPROM:M95256-WMN6P
- U1: footprint Package_QFP:LQFP-48_7x7mm_P0.5mm -> Housings_QFP:LQFP-48_7x7mm_Pitch0.5mm
Connections:
- net labels added: +3V3, +BATT, SPI1_CLK, SPI1_MISO, SPI1_MOSI, SYS_SWCLK, SYS_SWDIO, USART1_RX, USART1_TX, USB_DM, USB_DP, VDD, VDDA
- net labels removed: +3.3V
- wire segments 30 -> 88
Other:
- note added: "1.27mm ARM10 compatible"

Commit message: Smaller MCU updated schematics
Parts:
- removed C1, C3: 20pF, Resistors_SMD:R_0805_HandSoldering, symbol Device:C
- removed C11, C6, C7, C8, C9: 100nF, Capacitors_SMD:C_0805_HandSoldering, symbol Device:C
- removed C2, C4: 4.3pF, Resistors_SMD:R_0805_HandSoldering, symbol Device:C
- removed D1: RED, LEDs:LED_0805_HandSoldering, symbol Device:LED
- removed J1: Conn_ARM_JTAG_SWD_10, Pin_Headers:Pin_Header_Straight_2x05_Pitch1.27mm_SMD, symbol Connector:Conn_ARM_JTAG_SWD_10
- removed R2, R3: 10K, Resistors_SMD:R_0805_HandSoldering, symbol Device:R
- removed R4: 1K, Resistors_SMD:R_0805_HandSoldering, symbol Device:R
- removed R5: FBead, Resistors_SMD:R_0805_HandSoldering, symbol Device:R
- removed SW1: SW_Push, symbol Switch:SW_Push
- removed U1: STM32L053C8Tx, Housings_QFP:LQFP-48_7x7mm_Pitch0.5mm, symbol MCU_ST_STM32L0:STM32L053C8Tx
- removed Y1: 8MHz, Crystals:Crystal_SMD_HC49-SD_HandSoldering, symbol Device:Crystal
- removed Y2: 32.768kHz, symbol Device:Crystal
- renumbered C10 to C1, U2 to U1
Connections:
- net labels removed: RCC_OSC32_IN, RCC_OSC32_OUT, RCC_OSC_IN, RCC_OSC_OUT, SPI1_CLK, SPI1_MISO, SPI1_MOSI, SYS_SWCLK, SYS_SWDIO, USART1_RX, USART1_TX, USB_DM, USB_DP, VDDA, nRESET
- wire segments 88 -> 14
Other:
- note removed: "1.27mm ARM10 compatible"
- note removed: "ABS25-32.768KHz"
- moved on the sheet: C1

Commit message: Added temperature sensor
Connections:
- wire segments 14 -> 17
Changed lines of the file:
@@
 EESchema Schematic File Version 4
-LIBS:plant_sensor-cache
 EELAYER 26 0
 EELAYER END
 $Descr A4 11693 8268
 encoding utf-8
-Sheet 1 3
+Sheet 1 4
 Title "Overview"
 Date "2019-02-22"
@@
 $EndDescr
 $Sheet
-S 6700 2500 1900 1400
+S 6700 2500 700  1050
 U 5C6DADA9
 F0 "BLE" 50
@@
 	2150 2200 2150 2300
 $Sheet
-S 4850 2500 1450 1400
+S 4850 2500 1450 1800
 U 5C7262D1
 F0 "MCU" 50
@@
 F6 "BLE_IRQ" O R 6300 3250 50
 F7 "BLE_nRESET" O R 6300 3350 50
+F8 "TEMP_IRQ" I R 6300 4150 50
+F9 "I2C1_SCL" B R 6300 3900 50
+F10 "I2C1_SDA" B R 6300 4000 50
 $EndSheet
 Wire Wire Line
@@
 Wire Wire Line
 	6700 3350 6300 3350
+$Sheet
+S 6700 3750 700  550
+U 5C708F8B
+F0 "Temperature" 50
+F1 "plant_sensor-temp.sch" 50
+F2 "TEMP_SDA" B L 6700 3900 50
+F3 "TEMP_SCL" B L 6700 4000 50
+F4 "TEMP_IRQ" O L 6700 4150 50
+$EndSheet
+Wire Wire Line
+	6300 4000 6700 4000
+Wire Wire Line
+	6700 3900 6300 3900
+Wire Wire Line
+	6300 4150 6700 4150
 $EndSCHEMATC
