File: pcb/led_driver-light_sensor.sch (KiCad schematic (older format))
At the start: 2 parts, among them U5 TSL2550D

Commit message: ESP wroom module
Parts:
- C16: renamed from C1; footprint Capacitors_SMD:C_0805_HandSoldering -> Capacitor_SMD:C_0805_2012Metric_Pad1.15x1.40mm_HandSolder
- renumbered U5 to U3
Changed lines of the file:
@@
 EESchema Schematic File Version 4
 LIBS:rgb_controller-cache
-EELAYER 29 0
+EELAYER 30 0
 EELAYER END
 $Descr A4 11693 8268
 encoding utf-8
-Sheet 7 7
+Sheet 6 6
 Title "Light Sensor"
 Date "2019-02-23"
@@
 P 5600 3550
 AR Path="/5C7262D1/5C7F526E" Ref="U?"  Part="1"
-AR Path="/5C7F522E/5C7F526E" Ref="U5"  Part="1"
-F 0 "U5" H 5850 3200 50  0000 R CNN
+AR Path="/5C7F522E/5C7F526E" Ref="U3"  Part="1"
+F 0 "U3" H 5850 3200 50  0000 R CNN
 F 1 "TSL2550D" H 6150 3100 50  0000 R CNN
 F 2 "Housings_SOIC:SOIC-8_3.9x4.9mm_Pitch1.27mm" H 5600 3050 50  0001 C CNN
@@
 AR Path="/5C7F5275" Ref="#PWR?"  Part="1"
 AR Path="/5C7262D1/5C7F5275" Ref="#PWR?"  Part="1"
-AR Path="/5C7F522E/5C7F5275" Ref="#PWR0155"  Part="1"
-F 0 "#PWR0155" H 5600 3750 50  0001 C CNN
+AR Path="/5C7F522E/5C7F5275" Ref="#PWR070"  Part="1"
+F 0 "#PWR070" H 5600 3750 50  0001 C CNN
 F 1 "GND" H 5605 3827 50  0000 C CNN
 F 2 "" H 5600 4000 50  0001 C CNN
@@
 AR Path="/5C7F527D" Ref="#PWR?"  Part="1"
 AR Path="/5C7262D1/5C7F527D" Ref="#PWR?"  Part="1"
-AR Path="/5C7F522E/5C7F527D" Ref="#PWR0156"  Part="1"
-F 0 "#PWR0156" H 5600 3050 50  0001 C CNN
+AR Path="/5C7F522E/5C7F527D" Ref="#PWR069"  Part="1"
+F 0 "#PWR069" H 5600 3050 50  0001 C CNN
 F 1 "VDD" H 5617 3373 50  0000 C CNN
 F 2 "" H 5600 3200 50  0001 C CNN
@@
 AR Path="/5C7F5283" Ref="C?"  Part="1"
 AR Path="/5C7262D1/5C7F5283" Ref="C?"  Part="1"
-AR Path="/5C7F522E/5C7F5283" Ref="C1"  Part="1"
-F 0 "C1" H 5015 3746 50  0000 L CNN
+AR Path="/5C7F522E/5C7F5283" Ref="C16"  Part="1"
+F 0 "C16" H 5015 3746 50  0000 L CNN
 F 1 "100nF" H 5015 3655 50  0000 L CNN
-F 2 "Capacitors_SMD:C_0805_HandSoldering" H 4938 3550 50  0001 C CNN
+F 2 "Capacitor_SMD:C_0805_2012Metric_Pad1.15x1.40mm_HandSolder" H 4938 3550 50  0001 C CNN
 F 3 "~" H 4900 3700 50  0001 C CNN
 	1    4900 3700
@@
 AR Path="/5C7F528B" Ref="#PWR?"  Part="1"
 AR Path="/5C7262D1/5C7F528B" Ref="#PWR?"  Part="1"
-AR Path="/5C7F522E/5C7F528B" Ref="#PWR0157"  Part="1"
-F 0 "#PWR0157" H 4900 3750 50  0001 C CNN
+AR Path="/5C7F522E/5C7F528B" Ref="#PWR068"  Part="1"
+F 0 "#PWR068" H 4900 3750 50  0001 C CNN
 F 1 "GND" H 4905 3827 50  0000 C CNN
 F 2 "" H 4900 4000 50  0001 C CNN
@@
 AR Path="/5C7F5291" Ref="#PWR?"  Part="1"
 AR Path="/5C7262D1/5C7F5291" Ref="#PWR?"  Part="1"
-AR Path="/5C7F522E/5C7F5291" Ref="#PWR0158"  Part="1"
-F 0 "#PWR0158" H 4900 3050 50  0001 C CNN
+AR Path="/5C7F522E/5C7F5291" Ref="#PWR067"  Part="1"
+F 0 "#PWR067" H 4900 3050 50  0001 C CNN
 F 1 "VDD" H 4917 3373 50  0000 C CNN
 F 2 "" H 4900 3200 50  0001 C CNN
