File: pcb/led_driver-power.sch (KiCad schematic (older format))
At the start: 13 parts, among them IC5 LD1117S50TR_SOT223, IC6 LD3985M33R_SOT23, J3 Screw_Terminal_01x02

Commit message: dev
Parts:
- removed C14, C17: 1uF X5R, Capacitors_SMD:C_0805_HandSoldering, symbol Device:C
- removed C15, C18: 100nF, Capacitors_SMD:C_0805_HandSoldering, symbol Device:C
- removed C16: 10nF X7R, Capacitors_SMD:C_0805_HandSoldering, symbol Device:C
- removed D3, D4: MBR0520, Diodes_SMD:D_SOD-123, symbol Diode:MBR0520
- removed IC6: LD3985M33R_SOT23, TO_SOT_Packages_SMD:SOT-23-5_HandSoldering, symbol Regulator_Linear:LD3985M33R_SOT23
Connections:
- net labels added: +5V
- net labels removed: +3.3V, VBUS, VCOM
- wire segments 41 -> 14
