File: pcb/led_driver-power.sch (KiCad schematic (older format))
At the start: 13 parts, among them IC5 LD1117S50TR_SOT223, IC6 LD3985M33R_SOT23, J3 Screw_Terminal_01x02

Commit message: ESP wroom module
Parts:
- removed D3: MBR0520, Diodes_SMD:D_SOD-123, symbol Diode:MBR0520
- added C18: 15nF, Capacitor_SMD:C_0805_2012Metric_Pad1.15x1.40mm_HandSolder, symbol Device:C
- added D7: MMSZ5240BT1G, Diode_SMD:D_SOD-123, symbol Diode:MMSD914
- added Q5: IRF9540N, Package_TO_SOT_SMD:TO-263-2, symbol Transistor_FET:IRF9540N
- added R19: 10K, Resistor_SMD:R_0805_2012Metric_Pad1.15x1.40mm_HandSolder, symbol Device:R
- C10: renamed from C13; footprint Capacitors_Tantalum_SMD:CP_Tantalum_Case-C_EIA-6032-28_Hand -> Capacitor_Tantalum_SMD:CP_EIA-6032-28_Kemet-C_Pad2.25x2.35mm_HandSolder
- C11: renamed from C14; footprint Capacitors_SMD:C_0805_HandSoldering -> Capacitor_SMD:C_0805_2012Metric_Pad1.15x1.40mm_HandSolder
- C12: renamed from C15; footprint Capacitors_SMD:C_0805_HandSoldering -> Capacitor_SMD:C_0805_2012Metric_Pad1.15x1.40mm_HandSolder
- C13: renamed from C16; footprint Capacitors_SMD:C_0805_HandSoldering -> Capacitor_SMD:C_0805_2012Metric_Pad1.15x1.40mm_HandSolder
- C14: renamed from C17; footprint Capacitors_SMD:C_0805_HandSoldering -> Capacitor_SMD:C_0805_2012Metric_Pad1.15x1.40mm_HandSolder
- C15: renamed from C18; footprint Capacitors_SMD:C_0805_HandSoldering -> Capacitor_SMD:C_0805_2012Metric_Pad1.15x1.40mm_HandSolder
- C9: renamed from C12; footprint Capacitors_Tantalum_SMD:CP_Tantalum_Case-C_EIA-6032-28_Hand -> Capacitor_Tantalum_SMD:CP_EIA-6032-28_Kemet-C_Pad2.25x2.35mm_HandSolder
- renumbered D2 to D6, IC5 to IC3, IC6 to IC4, J3 to J4
Connections:
- net labels removed: VBUS
- wire segments 41 -> 47
Other:
- moved on the sheet: J4
