File: pcb/led_driver-power.sch (KiCad schematic (older format))
At the start: 16 parts, among them IC3 LD1117S50TR_SOT223, IC4 LD3985M33R_SOT23, J4 Screw_Terminal_01x02, Q5 IRF9540N

Commit message: backup
Parts:
- D4, D6: footprint Diodes_SMD:D_SOD-123 -> Diode_SMD:D_SOD-123
Changed lines of the file:
@@
 F 0 "D6" H 4250 3600 50  0000 C CNN
 F 1 "MBR0520" H 4150 3700 50  0000 C CNN
-F 2 "Diodes_SMD:D_SOD-123" H 4400 3475 50  0001 C CNN
+F 2 "Diode_SMD:D_SOD-123" H 4400 3475 50  0001 C CNN
 F 3 "http://www.mccsemi.com/up_pdf/MBR0520~MBR0580(SOD123).pdf" H 4400 3650 50  0001 C CNN
 	1    4400 3650
@@
 F 0 "D4" H 4250 2900 50  0000 C CNN
 F 1 "MBR0520" H 4150 3000 50  0000 C CNN
-F 2 "Diodes_SMD:D_SOD-123" H 4400 2775 50  0001 C CNN
+F 2 "Diode_SMD:D_SOD-123" H 4400 2775 50  0001 C CNN
 F 3 "http://www.mccsemi.com/up_pdf/MBR0520~MBR0580(SOD123).pdf" H 4400 2950 50  0001 C CNN
 	1    4400 2950
