File: pcb/rgb_controller-led-driver.sch (KiCad schematic (older format))
At the start: 17 parts, among them IC3 PM8834, IC4 PM8834, J4 Screw_Terminal_01x06, Q1 IRF3205SPBF, Q2 IRF3205SPBF, Q3 IRF3205SPBF, Q4 IRF3205SPBF

Commit message: Layouting and update
Parts:
- removed Q1, Q2, Q3, Q4: IRF3205SPBF, TO_SOT_Packages_SMD:TO-263-2, symbol IRF3205SPBF:IRF3205SPBF
- added Q1, Q2, Q3, Q4: IRF3205SPBF, TO_SOT_Packages_SMD:TO-263-2, symbol Transistor_FET:IRF3205
Connections:
- wire segments 60 -> 64
Changed lines of the file:
@@
 Comment2 ""
 Comment3 ""
-Comment4 ""
+Comment4 "Author: Sander Huisman"
 $EndDescr
 Text Label 2350 1450 0    50   ~ 0
@@
 	1    0    0    -1
 $EndComp
-$Comp
-L IRF3205SPBF:IRF3205SPBF Q1
-U 1 1 5C726DFF
-P 4500 3250
-AR Path="/5C726DFF" Ref="Q1"  Part="1"
-AR Path="/5C726A30/5C726DFF" Ref="Q1"  Part="1"
-F 0 "Q1" H 5050 3350 50  0000 L CNN
-F 1 "IRF3205SPBF" H 5050 3250 50  0000 L CNN
-F 2 "TO_SOT_Packages_SMD:TO-263-2" H 4500 3250 50  0001 L BNN
-F 3 "D2PAK Infineon" H 4500 3250 50  0001 L BNN
-F 4 "IRF3205SPBF" H 4500 3250 50  0001 L BNN "Field4"
-F 5 "None" H 4500 3250 50  0001 L BNN "Field5"
-F 6 "Infineon Technologies" H 4500 3250 50  0001 L BNN "Field6"
-F 7 "Single N-Channel 55 V 200 W 146 nC Hexfet Power Mosfet Surface Mount - D2PAK-3" H 4500 3250 50  0001 L BNN "Field7"
-F 8 "Unavailable" H 4500 3250 50  0001 L BNN "Field8"
-	1    4500 3250
-	1    0    0    -1
-$EndComp
-$Comp
-L IRF3205SPBF:IRF3205SPBF Q2
-U 1 1 5C726E75
-P 4800 3450
-AR Path="/5C726E75" Ref="Q2"  Part="1"
-AR Path="/5C726A30/5C726E75" Ref="Q2"  Part="1"
-F 0 "Q2" H 5050 3500 50  0000 L CNN
-F 1 "IRF3205SPBF" H 5050 3400 50  0000 L CNN
-F 2 "TO_SOT_Packages_SMD:TO-263-2" H 4800 3450 50  0001 L BNN
-F 3 "D2PAK Infineon" H 4800 3450 50  0001 L BNN
-F 4 "IRF3205SPBF" H 4800 3450 50  0001 L BNN "Field4"
-F 5 "None" H 4800 3450 50  0001 L BNN "Field5"
-F 6 "Infineon Technologies" H 4800 3450 50  0001 L BNN "Field6"
-F 7 "Single N-Channel 55 V 200 W 146 nC Hexfet Power Mosfet Surface Mount - D2PAK-3" H 4800 3450 50  0001 L BNN "Field7"
-F 8 "Unavailable" H 4800 3450 50  0001 L BNN "Field8"
-	1    4800 3450
-	1    0    0    -1
-$EndComp
 Wire Wire Line
 	4350 3350 4400 3350
 Wire Wire Line
-	4350 3550 4700 3550
-Wire Wire Line
-	4600 3450 4600 4000
-Wire Wire Line
-	4900 4000 4900 3650
+	4350 3550 4650 3550
+Wire Wire Line
+	4700 3550 4700 4000
+Wire Wire Line
+	5050 4000 5050 3800
 $Comp
 L power:GND #PWR0109
 U 1 1 5C72704A
-P 4600 4000
-F 0 "#PWR0109" H 4600 3750 50  0001 C CNN
-F 1 "GND" H 4605 3827 50  0000 C CNN
-F 2 "" H 4600 4000 50  0001 C CNN
-F 3 "" H 4600 4000 50  0001 C CNN
-	1    4600 4000
+P 4700 4000
+F 0 "#PWR0109" H 4700 3750 50  0001 C CNN
+F 1 "GND" H 4705 3827 50  0000 C CNN
+F 2 "" H 4700 4000 50  0001 C CNN
+F 3 "" H 4700 4000 50  0001 C CNN
+	1    4700 4000
 	1    0    0    -1
 $EndComp
@@
 L power:GND #PWR0110
 U 1 1 5C727078
-P 4900 4000
-F 0 "#PWR0110" H 4900 3750 50  0001 C CNN
-F 1 "GND" H 4905 3827 50  0000 C CNN
-F 2 "" H 4900 4000 50  0001 C CNN
-F 3 "" H 4900 4000 50  0001 C CNN
-	1    4900 4000
-	1    0    0    -1
-$EndComp
-Wire Wire Line
-	4900 3250 4900 2900
-Wire Wire Line
-	4600 2900 4600 3050
+P 5050 4000
+F 0 "#PWR0110" H 5050 3750 50  0001 C CNN
+F 1 "GND" H 5055 3827 50  0000 C CNN
+F 2 "" H 5050 4000 50  0001 C CNN
+F 3 "" H 5050 4000 50  0001 C CNN
+	1    5050 4000
+	1    0    0    -1
+$EndComp
 Wire Wire Line
 	3950 3950 3950 4000
@@
 	1    0    0    -1
 $EndComp
-$Comp
-L IRF3205SPBF:IRF3205SPBF Q3
-U 1 1 5C729B1F
-P 7850 3250
-AR Path="/5C729B1F" Ref="Q3"  Part="1"
-AR Path="/5C726A30/5C729B1F" Ref="Q3"  Part="1"
-F 0 "Q3" H 8400 3350 50  0000 L CNN
-F 1 "IRF3205SPBF" H 8400 3250 50  0000 L CNN
-F 2 "TO_SOT_Packages_SMD:TO-263-2" H 7850 3250 50  0001 L BNN
-F 3 "D2PAK Infineon" H 7850 3250 50  0001 L BNN
-F 4 "IRF3205SPBF" H 7850 3250 50  0001 L BNN "Field4"
-F 5 "None" H 7850 3250 50  0001 L BNN "Field5"
-F 6 "Infineon Technologies" H 7850 3250 50  0001 L BNN "Field6"
-F 7 "Single N-Channel 55 V 200 W 146 nC Hexfet Power Mosfet Surface Mount - D2PAK-3" H 7850 3250 50  0001 L BNN "Field7"
-F 8 "Unavailable" H 7850 3250 50  0001 L BNN "Field8"
-	1    7850 3250
-	1    0    0    -1
-$EndComp
-$Comp
-L IRF3205SPBF:IRF3205SPBF Q4
-U 1 1 5C729B2B
-P 8150 3450
-AR Path="/5C729B2B" Ref="Q4"  Part="1"
-AR Path="/5C726A30/5C729B2B" Ref="Q4"  Part="1"
-F 0 "Q4" H 8400 3500 50  0000 L CNN
-F 1 "IRF3205SPBF" H 8400 3400 50  0000 L CNN
-F 2 "TO_SOT_Packages_SMD:TO-263-2" H 8150 3450 50  0001 L BNN
-F 3 "D2PAK Infineon" H 8150 3450 50  0001 L BNN
-F 4 "IRF3205SPBF" H 8150 3450 50  0001 L BNN "Field4"
-F 5 "None" H 8150 3450 50  0001 L BNN "Field5"
-F 6 "Infineon Technologies" H 8150 3450 50  0001 L BNN "Field6"
-F 7 "Single N-Channel 55 V 200 W 146 nC Hexfet Power Mosfet Surface Mount - D2PAK-3" H 8150 3450 50  0001 L BNN "Field7"
-F 8 "Unavailable" H 8150 3450 50  0001 L BNN "Field8"
-	1    8150 3450
-	1    0    0    -1
-$EndComp
 Wire Wire Line
 	7700 3350 7750 3350
 Wire Wire Line
-	7700 3550 8050 3550
-Wire Wire Line
-	7950 3450 7950 4000
-Wire Wire Line
-	8250 4000 8250 3650
+	7700 3550 8000 3550
+Wire Wire Line
+	8050 3550 8050 4000
+Wire Wire Line
+	8400 4000 8400 3800
 $Comp
 L power:GND #PWR0117
 U 1 1 5C729B36
-P 7950 4000
-F 0 "#PWR0117" H 7950 3750 50  0001 C CNN
-F 1 "GND" H 7955 3827 50  0000 C CNN
-F 2 "" H 7950 4000 50  0001 C CNN
-F 3 "" H 7950 4000 50  0001 C CNN
-	1    7950 4000
+P 8050 4000
+F 0 "#PWR0117" H 8050 3750 50  0001 C CNN
+F 1 "GND" H 8055 3827 50  0000 C CNN
+F 2 "" H 8050 4000 50  0001 C CNN
+F 3 "" H 8050 4000 50  0001 C CNN
+	1    8050 4000
 	1    0    0    -1
 $EndComp
@@
 L power:GND #PWR0118
 U 1 1 5C729B3C
-P 8250 4000
-F 0 "#PWR0118" H 8250 3750 50  0001 C CNN
-F 1 "GND" H 8255 3827 50  0000 C CNN
-F 2 "" H 8250 4000 50  0001 C CNN
-F 3 "" H 8250 4000 50  0001 C CNN
-	1    8250 4000
-	1    0    0    -1
-$EndComp
-Wire Wire Line
-	8250 3250 8250 2900
-Wire Wire Line
-	7950 2900 7950 3050
+P 8400 4000
+F 0 "#PWR0118" H 8400 3750 50  0001 C CNN
+F 1 "GND" H 8405 3827 50  0000 C CNN
+F 2 "" H 8400 4000 50  0001 C CNN
+F 3 "" H 8400 4000 50  0001 C CNN
+	1    8400 4000
+	1    0    0    -1
+$EndComp
 Wire Wire Line
 	7300 3950 7300 4000
@@
 Wire Wire Line
 	8300 1550 8300 1500
-Text Label 4600 2900 1    50   ~ 0
+Text Label 4700 2900 1    50   ~ 0
 DRIVER_R
-Text Label 4900 2900 1    50   ~ 0
+Text Label 5050 2900 1    50   ~ 0
 DRIVER_G
-Text Label 7950 2900 1    50   ~ 0
+Text Label 8050 2900 1    50   ~ 0
 DRIVER_B
-Text Label 8250 2900 1    50   ~ 0
+Text Label 8400 2900 1    50   ~ 0
 DRIVER_W
 Text Label 7950 1950 0    50   ~ 0
@@
 Text Label 7950 1650 0    50   ~ 0
 DRIVER_W
+$Comp
+L Transistor_FET:IRF3205 Q1
+U 1 1 5C8DCC3C
+P 4600 3350
+F 0 "Q1" H 4805 3396 50  0000 L CNN
+F 1 "IRF3205SPBF" H 4805 3305 50  0000 L CNN
+F 2 "TO_SOT_Packages_SMD:TO-263-2" H 4850 3275 50  0001 L CIN
+F 3 "http://www.irf.com/product-info/datasheets/data/irf3205.pdf" H 4600 3350 50  0001 L CNN
+	1    4600 3350
+	1    0    0    -1
+$EndComp
+$Comp
+L Transistor_FET:IRF3205 Q2
+U 1 1 5C8DCE7F
+P 4950 3600
+F 0 "Q2" H 5155 3646 50  0000 L CNN
+F 1 "IRF3205SPBF" H 5155 3555 50  0000 L CNN
+F 2 "TO_SOT_Packages_SMD:TO-263-2" H 5200 3525 50  0001 L CIN
+F 3 "http://www.irf.com/product-info/datasheets/data/irf3205.pdf" H 4950 3600 50  0001 L CNN
+	1    4950 3600
+	1    0    0    -1
+$EndComp
+Wire Wire Line
+	4650 3550 4650 3600
+Wire Wire Line
+	4650 3600 4750 3600
+Wire Wire Line
+	4700 2900 4700 3150
+Wire Wire Line
+	5050 2900 5050 3400
+$Comp
+L Transistor_FET:IRF3205 Q3
+U 1 1 5C8E9AD6
+P 7950 3350
+F 0 "Q3" H 8155 3396 50  0000 L CNN
+F 1 "IRF3205SPBF" H 8155 3305 50  0000 L CNN
+F 2 "TO_SOT_Packages_SMD:TO-263-2" H 8200 3275 50  0001 L CIN
+F 3 "http://www.irf.com/product-info/datasheets/data/irf3205.pdf" H 7950 3350 50  0001 L CNN
+	1    7950 3350
+	1    0    0    -1
+$EndComp
+Wire Wire Line
+	8000 3550 8000 3600
+Wire Wire Line
+	8000 3600 8100 3600
+$Comp
+L Transistor_FET:IRF3205 Q4
+U 1 1 5C8EBAE1
+P 8300 3600
+F 0 "Q4" H 8505 3646 50  0000 L CNN
+F 1 "IRF3205SPBF" H 8505 3555 50  0000 L CNN
+F 2 "TO_SOT_Packages_SMD:TO-263-2" H 8550 3525 50  0001 L CIN
+F 3 "http://www.irf.com/product-info/datasheets/data/irf3205.pdf" H 8300 3600 50  0001 L CNN
+	1    8300 3600
+	1    0    0    -1
+$EndComp
+Wire Wire Line
+	8400 2900 8400 3400
+Wire Wire Line
+	8050 2900 8050 3150
 $EndSCHEMATC

Commit message: dev
Parts:
- C10, C11: footprint Capacitors_SMD:C_0805_HandSoldering -> Capacitor_SMD:C_0805_2012Metric_Pad1.15x1.40mm_HandSolder
- R10, R11, R12, R13, R6, R7, R8, R9: footprint Resistors_SMD:R_0805_HandSoldering -> Resistor_SMD:R_0805_2012Metric_Pad1.15x1.40mm_HandSolder
Changed lines of the file:
@@
 EESchema Schematic File Version 4
 LIBS:rgb_controller-cache
-EELAYER 29 0
+EELAYER 30 0
 EELAYER END
 $Descr A4 11693 8268
 encoding utf-8
-Sheet 5 7
+Sheet 4 6
 Title ""
 Date "2019-02-23"
@@
 F 0 "C10" H 5815 3846 50  0000 L CNN
 F 1 "1uF X7R" H 5815 3755 50  0000 L CNN
-F 2 "Capacitors_SMD:C_0805_HandSoldering" H 5738 3650 50  0001 C CNN
+F 2 "Capacitor_SMD:C_0805_2012Metric_Pad1.15x1.40mm_HandSolder" H 5738 3650 50  0001 C CNN
 F 3 "~" H 5700 3800 50  0001 C CNN
 	1    5700 3800
@@
 F 0 "R8" H 3470 2996 50  0000 L CNN
 F 1 "10K" H 3470 2905 50  0000 L CNN
-F 2 "Resistors_SMD:R_0805_HandSoldering" V 3330 2950 50  0001 C CNN
+F 2 "Resistor_SMD:R_0805_2012Metric_Pad1.15x1.40mm_HandSolder" V 3330 2950 50  0001 C CNN
 F 3 "~" H 3400 2950 50  0001 C CNN
 	1    3400 2950
@@
 F 0 "R6" H 3170 2996 50  0000 L CNN
 F 1 "10K" H 3170 2905 50  0000 L CNN
-F 2 "Resistors_SMD:R_0805_HandSoldering" V 3030 2950 50  0001 C CNN
+F 2 "Resistor_SMD:R_0805_2012Metric_Pad1.15x1.40mm_HandSolder" V 3030 2950 50  0001 C CNN
 F 3 "~" H 3100 2950 50  0001 C CNN
 	1    3100 2950
@@
 F 0 "C11" H 9165 3846 50  0000 L CNN
 F 1 "1uF X7R" H 9165 3755 50  0000 L CNN
-F 2 "Capacitors_SMD:C_0805_HandSoldering" H 9088 3650 50  0001 C CNN
+F 2 "Capacitor_SMD:C_0805_2012Metric_Pad1.15x1.40mm_HandSolder" H 9088 3650 50  0001 C CNN
 F 3 "~" H 9050 3800 50  0001 C CNN
 	1    9050 3800
@@
 F 0 "R11" H 6820 2996 50  0000 L CNN
 F 1 "10K" H 6820 2905 50  0000 L CNN
-F 2 "Resistors_SMD:R_0805_HandSoldering" V 6680 2950 50  0001 C CNN
+F 2 "Resistor_SMD:R_0805_2012Metric_Pad1.15x1.40mm_HandSolder" V 6680 2950 50  0001 C CNN
 F 3 "~" H 6750 2950 50  0001 C CNN
 	1    6750 2950
@@
 F 0 "R10" H 6520 2996 50  0000 L CNN
 F 1 "10K" H 6520 2905 50  0000 L CNN
-F 2 "Resistors_SMD:R_0805_HandSoldering" V 6380 2950 50  0001 C CNN
+F 2 "Resistor_SMD:R_0805_2012Metric_Pad1.15x1.40mm_HandSolder" V 6380 2950 50  0001 C CNN
 F 3 "~" H 6450 2950 50  0001 C CNN
 	1    6450 2950
@@
 F 0 "R9" H 3470 3796 50  0000 L CNN
 F 1 "10K" H 3470 3705 50  0000 L CNN
-F 2 "Resistors_SMD:R_0805_HandSoldering" V 3330 3750 50  0001 C CNN
+F 2 "Resistor_SMD:R_0805_2012Metric_Pad1.15x1.40mm_HandSolder" V 3330 3750 50  0001 C CNN
 F 3 "~" H 3400 3750 50  0001 C CNN
 	1    3400 3750
@@
 F 0 "R7" H 3170 3796 50  0000 L CNN
 F 1 "10K" H 3170 3705 50  0000 L CNN
-F 2 "Resistors_SMD:R_0805_HandSoldering" V 3030 3750 50  0001 C CNN
+F 2 "Resistor_SMD:R_0805_2012Metric_Pad1.15x1.40mm_HandSolder" V 3030 3750 50  0001 C CNN
 F 3 "~" H 3100 3750 50  0001 C CNN
 	1    3100 3750
@@
 F 0 "R13" H 6820 3796 50  0000 L CNN
 F 1 "10K" H 6820 3705 50  0000 L CNN
-F 2 "Resistors_SMD:R_0805_HandSoldering" V 6680 3750 50  0001 C CNN
+F 2 "Resistor_SMD:R_0805_2012Metric_Pad1.15x1.40mm_HandSolder" V 6680 3750 50  0001 C CNN
 F 3 "~" H 6750 3750 50  0001 C CNN
 	1    6750 3750
@@
 F 0 "R12" H 6520 3796 50  0000 L CNN
 F 1 "10K" H 6520 3705 50  0000 L CNN
-F 2 "Resistors_SMD:R_0805_HandSoldering" V 6380 3750 50  0001 C CNN
+F 2 "Resistor_SMD:R_0805_2012Metric_Pad1.15x1.40mm_HandSolder" V 6380 3750 50  0001 C CNN
 F 3 "~" H 6450 3750 50  0001 C CNN
 	1    6450 3750
