File: pcb/rgb_controller-mcu.sch (KiCad schematic (older format))
At the start: 39 parts, among them IC2 STM32L052K8Tx, J1 Conn_ARM_JTAG_SWD_10, J2 COM, J5 USB_B_Micro, J6 Screw_Terminal_01x04, Q6 BSS138, SW1 SW_Push, U3 USBLC6-2SC6, U4 CCS811, U7 BME280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

Commit message: dev
Parts:
- removed C3, C4, C5, C8: 100nF, Capacitors_SMD:C_0805_HandSoldering, symbol Device:C
- removed C6, C7: 4.3pF, Capacitors_SMD:C_0805_HandSoldering, symbol Device:C
- removed IC2: STM32L052K8Tx, Housings_QFP:LQFP-32_7x7mm_Pitch0.8mm, symbol MCU_ST_STM32L0:STM32L052K8Tx
- removed J1: Conn_ARM_JTAG_SWD_10, Pin_Headers:Pin_Header_Straight_2x05_Pitch1.27mm_SMD, symbol Connector:Conn_ARM_JTAG_SWD_10
- removed J2: COM, Pin_Headers:Pin_Header_Straight_1x06_Pitch2.54mm, symbol Connector:Conn_01x06_Male
- removed J5: USB_B_Micro, Connectors:USB_Micro-B, symbol Connector:USB_B_Micro
- removed Q6: BSS138, TO_SOT_Packages_SMD:SOT-23_Handsoldering, symbol Transistor_FET:BSS138
- removed R14: 100K, Resistors_SMD:R_0805_HandSoldering, symbol Device:R
- removed R15: 1K5, Resistors_SMD:R_0805_HandSoldering, symbol Device:R
- removed R16, R3, R4: 10K, Resistors_SMD:R_0805_HandSoldering, symbol Device:R
- removed R17: 36K, Resistors_SMD:R_0805_HandSoldering, symbol Device:R
- removed R18: 100, Resistors_SMD:R_0805_HandSoldering, symbol Device:R
- removed R2: FBead, Resistors_SMD:R_0805_HandSoldering, symbol Device:R
- removed SW1: SW_Push, Button_Switch_SMD:SW_SPST_B3S-1000, symbol Switch:SW_Push
- removed U3: USBLC6-2SC6, TO_SOT_Packages_SMD:SOT-23-6_Handsoldering, symbol Power_Protection:USBLC6-2SC6
- removed U4: CCS811, Package_LGA:AMS_LGA-10-1EP_2.7x4mm_P0.6mm, symbol Sensor_Gas:CCS811
- removed U7: BME280, Package_LGA:Bosch_LGA-8_2.5x2.5mm_P0.65mm_ClockwisePinNumbering, symbol Sensor:BME280
- removed Y1: 32.768kHz, symbol Device:Crystal
- added U1: WeMos_D1_mini, Module:WEMOS_D1_mini_light, symbol MCU_Module:WeMos_D1_mini
- C19, C20: footprint Capacitors_SMD:C_0805_HandSoldering -> Capacitor_SMD:C_0805_2012Metric_Pad1.15x1.40mm_HandSolder
- R19, R20, R5: footprint Resistors_SMD:R_0805_HandSoldering -> Resistor_SMD:R_0805_2012Metric_Pad1.15x1.40mm_HandSolder
Connections:
- net labels added: +3V3, +5V
- net labels removed: BLE_IRQ, BLE_nCS, BLE_nRESET, RCC_OSC32_IN, RCC_OSC32_OUT, RXD, SPI1_CLK, SPI1_MISO, SPI1_MOSI, SYS_SWCLK, SYS_SWDIO, TEMP_IRQ, TXD, USB_D+, USB_D-, USB_RENUMn, VBUS, VCOM, VDDA, nRESET
- wire segments 162 -> 53
- no-connect marks 2 -> 0
Other:
- note removed: "1.27mm ARM10 compatible"
- note removed: "5V"
- note removed: "ABS25-32.768KHz"
- note removed: "CTS"
- note removed: "RTS"
- note removed: "TTL-232R-3V3 compatible"
- moved on the sheet: R19, R20
