File: pcb/rgb_controller-mcu.sch (KiCad schematic (older format))
At the start: 16 parts, among them IC2 STM32L052K8Tx, J1 Conn_ARM_JTAG_SWD_10, J2 COM, SW1 SW_Push, Y1 32.768kHz

Commit message: WIP
Parts:
- added J5: USB_B_Micro, Connectors:USB_Micro-B, symbol Connector:USB_B_Micro
- added Q6: BSS138, TO_SOT_Packages_SMD:SOT-23_Handsoldering, symbol Transistor_FET:BSS138
- added R14: 100K, Resistors_SMD:R_0805_HandSoldering, symbol Device:R
- added R15: 1K5, Resistors_SMD:R_0805_HandSoldering, symbol Device:R
- added R16: 10K, Resistors_SMD:R_0805_HandSoldering, symbol Device:R
- added R17: 36K, Resistors_SMD:R_0805_HandSoldering, symbol Device:R
- added R18: 100, Resistors_SMD:R_0805_HandSoldering, symbol Device:R
- added R19, R20: 4K7, Resistors_SMD:R_0805_HandSoldering, symbol Device:R
- added U3: USBLC6-2SC6, TO_SOT_Packages_SMD:SOT-23-6_Handsoldering, symbol Power_Protection:USBLC6-2SC6
- added U4: CCS811, Package_LGA:AMS_LGA-10-1EP_2.7x4mm_P0.6mm, symbol Sensor_Gas:CCS811
- added U7: BME280, Package_LGA:Bosch_LGA-8_2.5x2.5mm_P0.65mm_ClockwisePinNumbering, symbol Sensor:BME280
- C6, C7: footprint Resistors_SMD:R_0805_HandSoldering -> Capacitors_SMD:C_0805_HandSoldering
- J2: footprint Pin_Headers:Pin_Header_Angled_1x06_Pitch2.54mm -> Pin_Headers:Pin_Header_Straight_1x06_Pitch2.54mm
Connections:
- net labels added: LED_B, LED_G, LED_R, LED_W, USB_D+, USB_D-, USB_RENUMn, VCOM
- net labels removed: USB_DM, USB_DP
- wire segments 79 -> 128
Other:
- note removed: "USB?"
- moved on the sheet: C6, C7, J2

Commit message: Layouting
Parts:
- SW1: footprint (none) -> Button_Switch_SMD:SW_SPST_B3S-1000
Connections:
- wire segments 128 -> 130
Changed lines of the file:
@@
 EESchema Schematic File Version 4
-LIBS:rgb_controller-cache
-EELAYER 26 0
+EELAYER 29 0
 EELAYER END
 $Descr A4 11693 8268
@@
 F 0 "SW1" V 8354 5598 50  0000 L CNN
 F 1 "SW_Push" V 8445 5598 50  0000 L CNN
-F 2 "" H 8400 5650 50  0001 C CNN
+F 2 "Button_Switch_SMD:SW_SPST_B3S-1000" H 8400 5650 50  0001 C CNN
 F 3 "" H 8400 5650 50  0001 C CNN
 	1    8400 5450
@@
 L Sensor_Gas:CCS811 U4
 U 1 1 5C7A0E9F
-P 17900 2550
-F 0 "U4" H 17900 3228 50  0000 C CNN
-F 1 "CCS811" H 17900 3137 50  0000 C CNN
-F 2 "Package_LGA:AMS_LGA-10-1EP_2.7x4mm_P0.6mm" H 17900 1950 50  0001 C CNN
-F 3 "http://ams.com/eng/Products/Environmental-Sensors/Air-Quality-Sensors/CCS811" H 17900 2350 50  0001 C CNN
-	1    17900 2550
+P 17000 2750
+F 0 "U4" H 17000 3428 50  0000 C CNN
+F 1 "CCS811" H 17000 3337 50  0000 C CNN
+F 2 "Package_LGA:AMS_LGA-10-1EP_2.7x4mm_P0.6mm" H 17000 2150 50  0001 C CNN
+F 3 "http://ams.com/eng/Products/Environmental-Sensors/Air-Quality-Sensors/CCS811" H 17000 2550 50  0001 C CNN
+	1    17000 2750
 	1    0    0    -1
 $EndComp
@@
 L Sensor:BME280 U7
 U 1 1 5C7A1D5A
-P 19150 2500
-F 0 "U7" H 18720 2546 50  0000 R CNN
-F 1 "BME280" H 18720 2455 50  0000 R CNN
-F 2 "Package_LGA:Bosch_LGA-8_2.5x2.5mm_P0.65mm_ClockwisePinNumbering" H 19150 2300 50  0001 C CNN
-F 3 "https://ae-bst.resource.bosch.com/media/_tech/media/datasheets/BST-BME280_DS001-11.pdf" H 19150 2300 50  0001 C CNN
-	1    19150 2500
+P 18250 2700
+F 0 "U7" H 17820 2746 50  0000 R CNN
+F 1 "BME280" H 17820 2655 50  0000 R CNN
+F 2 "Package_LGA:Bosch_LGA-8_2.5x2.5mm_P0.65mm_ClockwisePinNumbering" H 18250 2500 50  0001 C CNN
+F 3 "https://ae-bst.resource.bosch.com/media/_tech/media/datasheets/BST-BME280_DS001-11.pdf" H 18250 2500 50  0001 C CNN
+	1    18250 2700
 	1    0    0    -1
 $EndComp
@@
 Wire Wire Line
 	6200 3500 6750 3500
-Text Label 6750 3500 0    50   ~ 0
+Text Label 6750 4200 0    50   ~ 0
 USB_RENUMn
 Text Label 4500 4100 0    50   ~ 0
@@
 Text Label 4500 4200 0    50   ~ 0
 I2C1_SDA
+Wire Wire Line
+	6200 3100 6750 3100
+Text Label 6750 3100 0    50   ~ 0
+BLE_nCS
+Wire Wire Line
+	6200 4200 6750 4200
+Text Label 6750 3500 0    50   ~ 0
+BLE_IRQ
 $EndSCHEMATC

Commit message: layouting
Parts:
- added C19, C20: 100nF, Capacitors_SMD:C_0805_HandSoldering, symbol Device:C
- added D5, D6: BAT54S, Package_TO_SOT_SMD:SOT-23, symbol Diode:BAT54S
- added J6: Screw_Terminal_01x04, TerminalBlock_Phoenix:TerminalBlock_Phoenix_PT-1,5-4-3.5-H_1x04_P3.50mm_Horizontal, symbol Connector:Screw_Terminal_01x04
- added R22, R25: 10R, Resistor_SMD:R_0805_2012Metric_Pad1.15x1.40mm_HandSolder, symbol Device:R
- added R23, R26: 1K, Resistor_SMD:R_0805_2012Metric_Pad1.15x1.40mm_HandSolder, symbol Device:R
- added R24, R27: 10K, Resistor_SMD:R_0805_2012Metric_Pad1.15x1.40mm_HandSolder, symbol Device:R
Connections:
- wire segments 130 -> 162

Commit message: ESP wroom module
Parts:
- removed C3, C5: 100nF, Capacitors_SMD:C_0805_HandSoldering, symbol Device:C
- removed C6, C7: 4.3pF, Capacitors_SMD:C_0805_HandSoldering, symbol Device:C
- removed IC2: STM32L052K8Tx, Housings_QFP:LQFP-32_7x7mm_Pitch0.8mm, symbol MCU_ST_STM32L0:STM32L052K8Tx
- removed J1: Conn_ARM_JTAG_SWD_10, Pin_Headers:Pin_Header_Straight_2x05_Pitch1.27mm_SMD, symbol Connector:Conn_ARM_JTAG_SWD_10
- removed J5: USB_B_Micro, Connectors:USB_Micro-B, symbol Connector:USB_B_Micro
- removed Q6: BSS138, TO_SOT_Packages_SMD:SOT-23_Handsoldering, symbol Transistor_FET:BSS138
- removed R14: 100K, Resistors_SMD:R_0805_HandSoldering, symbol Device:R
- removed R15: 1K5, Resistors_SMD:R_0805_HandSoldering, symbol Device:R
- removed R16, R3: 10K, Resistors_SMD:R_0805_HandSoldering, symbol Device:R
- removed R17: 36K, Resistors_SMD:R_0805_HandSoldering, symbol Device:R
- removed R19, R20: 4K7, Resistors_SMD:R_0805_HandSoldering, symbol Device:R
- removed R2: FBead, Resistors_SMD:R_0805_HandSoldering, symbol Device:R
- removed U3: USBLC6-2SC6, TO_SOT_Packages_SMD:SOT-23-6_Handsoldering, symbol Power_Protection:USBLC6-2SC6
- removed U4: CCS811, Package_LGA:AMS_LGA-10-1EP_2.7x4mm_P0.6mm, symbol Sensor_Gas:CCS811
- removed U7: BME280, Package_LGA:Bosch_LGA-8_2.5x2.5mm_P0.65mm_ClockwisePinNumbering, symbol Sensor:BME280
- removed Y1: 32.768kHz, symbol Device:Crystal
- added C17: 100nF, Capacitor_SMD:C_0805_2012Metric_Pad1.15x1.40mm_HandSolder, symbol Device:C
- added C2: 10uF, Capacitor_Tantalum_SMD:CP_EIA-6032-28_Kemet-C_Pad2.25x2.35mm_HandSolder, symbol Device:CP
- added SW2: SW_Push, Button_Switch_SMD:SW_SPST_B3S-1000, symbol Switch:SW_Push
- added U1: ESP32-WROOM-32D, RF_Module:ESP32-WROOM-32, symbol RF_Module:ESP32-WROOM-32D
- C1: renamed from C4; footprint Capacitors_SMD:C_0805_HandSoldering -> Capacitor_SMD:C_0805_2012Metric_Pad1.15x1.40mm_HandSolder
- C3: renamed from C19; footprint Capacitors_SMD:C_0805_HandSoldering -> Capacitor_SMD:C_0805_2012Metric_Pad1.15x1.40mm_HandSolder
- C4: renamed from C20; footprint Capacitors_SMD:C_0805_HandSoldering -> Capacitor_SMD:C_0805_2012Metric_Pad1.15x1.40mm_HandSolder
- C5: renamed from C8; footprint Capacitors_SMD:C_0805_HandSoldering -> Capacitor_SMD:C_0805_2012Metric_Pad1.15x1.40mm_HandSolder
- R18: value 100 -> 10K; footprint Resistors_SMD:R_0805_HandSoldering -> Resistor_SMD:R_0805_2012Metric_Pad1.15x1.40mm_HandSolder
- R7: renamed from R4; footprint Resistors_SMD:R_0805_HandSoldering -> Resistor_SMD:R_0805_2012Metric_Pad1.15x1.40mm_HandSolder
- R8: renamed from R5; footprint Resistors_SMD:R_0805_HandSoldering -> Resistor_SMD:R_0805_2012Metric_Pad1.15x1.40mm_HandSolder
- renumbered D5 to D1, D6 to D2, D1 to D3, J6 to J1, R22 to R1, R23 to R2, R24 to R3, R25 to R4, R26 to R5, R27 to R6
Connections:
- net labels added: EN, I2C_SCL, I2C_SDA, IO0, IO13, RXD0, TXD0
- net labels removed: BLE_IRQ, BLE_nCS, BLE_nRESET, LED, RCC_OSC32_IN, RCC_OSC32_OUT, SPI1_CLK, SPI1_MISO, SPI1_MOSI, SYS_SWCLK, SYS_SWDIO, TEMP_IRQ, USART1_RX, USART1_TX, USB_D+, USB_D-, USB_RENUMn, VBUS, VDDA, nRESET
- wire segments 162 -> 78
Other:
- note removed: "1.27mm ARM10 compatible"
- note removed: "ABS25-32.768KHz"
- moved on the sheet: C1, C5, D3, R7, R8, SW1

Commit message: backup
Connections:
- net labels added: IN1, IN2
Other:
- moved on the sheet: C3, C4, D1, D2, J1, R1, R2, R3, R4, R5, R6
