File: pcb/rgb_controller.kicad_pcb (KiCad board)
At the start: 2 copper layers, 23 parts, among them IC1 SPBTLE-RF0, IC2 STM32L052K8Tx, J1 Conn_ARM_JTAG_SWD_10, J2 COM, U1 M95256-WMN6P, U2 LM75B, Y1 32.768kHz

Commit message: WIP
Parts:
- removed BT1: CR2032, Connectors:CR2032H
- removed U1: M95256-WMN6P, Housings_SOIC:SOIC-8_3.9x4.9mm_Pitch1.27mm
- added C10: 1uF X7R, Capacitors_SMD:C_0805_HandSoldering, F.Cu at (101.1, 144.3)
- added C11: 1uF X7R, Capacitors_SMD:C_0805_HandSoldering, F.Cu at (93.0, 144.3)
- added C12: 10uF, Capacitors_Tantalum_SMD:CP_Tantalum_Case-C_EIA-6032-28_Hand, F.Cu at (88.4, 174.0)
- added C13: 10uF, Capacitors_Tantalum_SMD:CP_Tantalum_Case-C_EIA-6032-28_Hand, F.Cu at (76.7, 174.0)
- added C14: 1uF X5R, Capacitors_SMD:C_0805_HandSoldering, F.Cu at (87.9, 146.6)
- added C15: 100nF, Capacitors_SMD:C_0805_HandSoldering, F.Cu at (85.9, 146.6)
- added C16: 10nF X7R, Capacitors_SMD:C_0805_HandSoldering, F.Cu at (82.8, 143.0)
- added C17: 1uF X5R, Capacitors_SMD:C_0805_HandSoldering, F.Cu at (77.7, 146.6)
- added C18: 100nF, Capacitors_SMD:C_0805_HandSoldering, F.Cu at (79.8, 146.6)
- added D2: MBR0520, Diodes_SMD:D_SOD-123, F.Cu at (76.2, 163.8)
- added D3: MBR0520, Diodes_SMD:D_SOD-123, F.Cu at (77.7, 140.2)
- added D4: MBR0520, Diodes_SMD:D_SOD-123, F.Cu at (77.7, 142.7)
- added IC3: PM8834, Housings_SOIC:SOIC-8_3.9x4.9mm_Pitch1.27mm, F.Cu at (105.2, 144.5)
- added IC4: PM8834, Housings_SOIC:SOIC-8_3.9x4.9mm_Pitch1.27mm, F.Cu at (97.0, 144.5)
- added IC5: LD1117S50TR_SOT223, TO_SOT_Packages_SMD:SOT-223-3_TabPin2, F.Cu at (82.5, 174.8)
- added IC6: LD3985M33R_SOT23, TO_SOT_Packages_SMD:SOT-23-5_HandSoldering, F.Cu at (82.8, 146.6)
- added J3: Screw_Terminal_01x02, Connectors_Phoenix:PhoenixContact_MC-G_02x3.50mm_Angled, F.Cu at (93.7, 171.4)
- added J4: Screw_Terminal_01x06, Connectors_Phoenix:PhoenixContact_MC-G_06x3.50mm_Angled, F.Cu at (103.4, 171.4)
- added J5: USB_B_Micro, Connectors:USB_Micro-B, F.Cu at (78.4, 134.1)
- added Q1: IRF3205SPBF, TO_SOT_Packages_SMD:TO-263-2, F.Cu at (117.6, 157.7)
- added Q2: IRF3205SPBF, TO_SOT_Packages_SMD:TO-263-2, F.Cu at (106.2, 157.7)
- added Q3: IRF3205SPBF, TO_SOT_Packages_SMD:TO-263-2, F.Cu at (94.7, 157.7)
- added Q4: IRF3205SPBF, TO_SOT_Packages_SMD:TO-263-2, F.Cu at (83.3, 157.7)
- added Q6: BSS138, TO_SOT_Packages_SMD:SOT-23_Handsoldering, F.Cu at (87.1, 138.5)
- added R10: 10K, Resistors_SMD:R_0805_HandSoldering, F.Cu at (101.3, 138.2)
- added R11: 10K, Resistors_SMD:R_0805_HandSoldering, F.Cu at (99.3, 138.2)
- added R12: 10K, Resistors_SMD:R_0805_HandSoldering, F.Cu at (95.2, 138.2)
- added R13: 10K, Resistors_SMD:R_0805_HandSoldering, F.Cu at (97.3, 138.2)
- added R14: 100K, Resistors_SMD:R_0805_HandSoldering, F.Cu at (82.3, 138.2)
- added R15: 1K5, Resistors_SMD:R_0805_HandSoldering, F.Cu at (84.3, 138.2)
- added R16: 10K, Resistors_SMD:R_0805_HandSoldering, F.Cu at (91.7, 138.2)
- added R17: 36K, Resistors_SMD:R_0805_HandSoldering, F.Cu at (89.9, 138.2)
- added R18: 100, Resistors_SMD:R_0805_HandSoldering, F.Cu at (91.9, 132.8)
- added R19: 4K7, Resistors_SMD:R_0805_HandSoldering, F.Cu at (152.4, 128.0)
- added R20: 4K7, Resistors_SMD:R_0805_HandSoldering, F.Cu at (152.4, 126.0)
- added R21: 10K, Resistors_SMD:R_0805_HandSoldering, F.Cu at (117.9, 138.2)
- added R6: 10K, Resistors_SMD:R_0805_HandSoldering, F.Cu at (109.5, 138.2)
- added R7: 10K, Resistors_SMD:R_0805_HandSoldering, F.Cu at (103.4, 138.2)
- added R8: 10K, Resistors_SMD:R_0805_HandSoldering, F.Cu at (107.4, 138.2)
- added R9: 10K, Resistors_SMD:R_0805_HandSoldering, F.Cu at (105.4, 138.2)
- added U3: USBLC6-2SC6, TO_SOT_Packages_SMD:SOT-23-6_Handsoldering, F.Cu at (83.8, 133.8)
- added U5: TSL2550D, Housings_SOIC:SOIC-8_3.9x4.9mm_Pitch1.27mm, F.Cu at (111.0, 144.5)
- C1: value 1uF X5R -> 100nF
- C6, C7: footprint Resistors_SMD:R_0805_HandSoldering -> Capacitors_SMD:C_0805_HandSoldering
- C9: footprint Capacitor_SMD:C_0805_2012Metric_Pad1.15x1.40mm_HandSolder -> Capacitors_SMD:C_0805_HandSoldering
- J2: footprint Pin_Headers:Pin_Header_Angled_1x06_Pitch2.54mm -> Pin_Headers:Pin_Header_Straight_1x06_Pitch2.54mm
- moved C8 117.3 mm to (158.8, 113.3)
- moved R4 114.8 mm to (138.3, 126.2)
- moved C1 101.7 mm to (114.8, 144.5), turned to 270 degrees
- moved R1 96.6 mm to (135.9, 108.3), turned to 270 degrees
- moved C9 53.5 mm to (122.4, 144.5), turned to 90 degrees
- moved C2 53.4 mm to (137.9, 108.2), turned to 270 degrees
- moved IC1 52.4 mm to (146.8, 106.9)
- moved J1 50.6 mm to (138.8, 121.2)
- moved C3 50.2 mm to (141.0, 112.0), turned to 180 degrees
- moved J2 48.8 mm to (132.6, 120.9)
- moved R2 48.5 mm to (158.8, 119.1)
- moved C4 48.5 mm to (158.8, 121.2)
- moved C5 48.5 mm to (158.8, 117.1)
- moved R3 48.5 mm to (158.8, 123.2)
- moved C6 47.8 mm to (174.2, 124.6)
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Connections:
- C1 pad 1: +BATT -> +3V3
- IC2 pad 18: Net-(IC2-Pad18) -> /MCU/USB_RENUMn
- IC2 pad 21: /MCU/USB_DM -> /MCU/USB_D-
- IC2 pad 22: /MCU/USB_DP -> /MCU/USB_D+
- IC2 pad 6: Net-(IC2-Pad6) -> /LED driver/LED_R
- IC2 pad 7: Net-(IC2-Pad7) -> /LED driver/LED_G
- IC2 pad 8: Net-(IC2-Pad8) -> /LED driver/LED_B
- IC2 pad 9: Net-(IC2-Pad9) -> /LED driver/LED_W
- J2 pad 3: VBUS -> VCOM
- U2 pad 1: /MCU/I2C1_SCL -> /MCU/I2C1_SDA
- U2 pad 2: /MCU/I2C1_SDA -> /MCU/I2C1_SCL
Routing:
- net /LED driver/DRIVER_W: track 0.00 -> 20.8 mm
- net /LED driver/DRIVER_B: track 0.00 -> 13.5 mm
- net +12V: track 0.00 -> 6.13 mm
- net /LED driver/DRIVER_R: track 0.00 -> 6.03 mm
- net /MCU/USB_D+: track 0.00 -> 5.69 mm
- net /MCU/USB_D-: track 0.00 -> 5.66 mm
- net Net-(J5-Pad4): track 0.00 -> 4.17 mm
- net /LED driver/DRIVER_G: track 0.00 -> 3.25 mm
- net /LED driver/LED_B: track 0.00 -> 2.46 mm
- net Net-(IC4-Pad1): track 0.00 -> 2.46 mm
- net /LED driver/LED_R: track 0.00 -> 2.38 mm
- net Net-(IC3-Pad1): track 0.00 -> 2.38 mm
- net /LED driver/LED_W: track 0.00 -> 2.35 mm
- net /LED driver/LED_G: track 0.00 -> 2.27 mm
- net VBUS: track 0.00 -> 1.47 mm, vias 0 -> 1
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- added copper zone on F.Cu, net GND
Other:
- board outline added: 50 x 80 mm
- board text added: "12V"
- board text added: "B"
- board text added: "G"
- board text added: "GND"
- board text added: "R"
- board text added: "W"

Commit message: Layouting and update
Parts:
- moved R1 221.9 mm to (357.1, 125.8)
- moved J1 221.9 mm to (359.9, 138.6)
- moved R4 221.9 mm to (359.5, 143.7)
- moved C3 221.9 mm to (362.2, 129.5)
- moved C8 221.9 mm to (379.9, 130.7)
- moved IC1 221.9 mm to (368.0, 124.4)
- moved R2 221.9 mm to (379.9, 136.6)
- moved R3 221.9 mm to (379.9, 140.7)
- moved Y1 221.9 mm to (389.8, 134.3)
- moved C4 221.9 mm to (379.9, 138.6)
- moved C5 221.9 mm to (379.9, 134.6)
- moved C6 221.9 mm to (395.4, 142.1)
- moved C7 221.9 mm to (395.4, 128.6)
- moved IC2 221.9 mm to (369.8, 133.8)
- moved R19 221.9 mm to (373.6, 145.5)
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Routing:
- net +12V: track 6.13 -> 65.9 mm, vias 0 -> 3
- net Net-(IC3-Pad7): track 0.00 -> 19.4 mm
- net Net-(C13-Pad1): track 0.00 -> 19.3 mm
- net Net-(IC4-Pad5): track 0.00 -> 14.3 mm
- net Net-(IC3-Pad5): track 0.00 -> 10.8 mm
- net /LED driver/DRIVER_W: track 20.8 -> 31.4 mm
- net Net-(IC4-Pad8): track 0.00 -> 8.49 mm, vias 0 -> 2
- net Net-(IC3-Pad8): track 0.00 -> 8.49 mm, vias 0 -> 2
- net /LED driver/DRIVER_G: track 3.25 -> 9.37 mm
- net +3V3: track 0.00 -> 5.86 mm
- net Net-(IC4-Pad7): track 0.00 -> 5.76 mm
- net /MCU/USB_D+: track 5.69 -> 0.00 mm
- net /MCU/USB_D-: track 5.66 -> 0.00 mm
- net Net-(J5-Pad4): track 4.17 -> 0.00 mm
- net /LED driver/DRIVER_R: track 6.03 -> 10.0 mm
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Other:
- board size 50 x 80 mm -> 50 x 75 mm
- net class Default: clearance 0.2 -> 0.2032; trace_width 0.25 -> 0.2032; via_dia 0.8 -> 0.762; via_drill 0.4 -> 0.381
- rule trace_clearance: 0.2 -> 0.2032
- rule trace_min: 0.2 -> 0.1524
- rule via_min_drill: 0.3 -> 0.254
- rule via_min_size: 0.4 -> 0.508

Commit message: Layouting
Parts:
- added SW1: SW_Push, Button_Switch_SMD:SW_SPST_B3S-1100, F.Cu at (205.4, 105.1)
- moved C6 153.2 mm to (243.2, 125.1), turned to 270 degrees
- moved J1 152.7 mm to (208.3, 120.7)
- moved C7 152.4 mm to (243.2, 120.7), turned to 90 degrees
- moved J2 152.4 mm to (201.9, 122.6)
- moved R3 150.4 mm to (230.2, 127.0)
- moved R4 147.5 mm to (213.7, 121.9), turned to 270 degrees
- moved C5 147.0 mm to (234.0, 117.2)
- moved R2 147.0 mm to (234.0, 119.1), turned to 180 degrees
- moved C4 146.7 mm to (234.0, 124.1)
- moved C8 146.3 mm to (234.0, 121.0)
- moved C2 146.2 mm to (213.4, 113.3), turned to 180 degrees
- moved IC1 144.7 mm to (223.8, 111.4)
- moved R1 144.5 mm to (213.4, 111.4), turned to 180 degrees
- moved C3 144.0 mm to (218.8, 116.5)
- moved IC2 144.0 mm to (226.4, 120.7)
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Connections:
- IC2 pad 10: Net-(IC2-Pad10) -> /BLE/BLE_nCS
- IC2 pad 18: /MCU/USB_RENUMn -> /BLE/BLE_IRQ
- IC2 pad 25: Net-(IC2-Pad25) -> /MCU/USB_RENUMn
Routing:
- net +3V3: track 5.86 -> 77.7 mm, vias 0 -> 7
- net /MCU/I2C1_SDA: track 0.00 -> 34.2 mm, vias 0 -> 4
- net /MCU/I2C1_SCL: track 0.00 -> 33.3 mm, vias 0 -> 4
- net VCOM: track 0.00 -> 28.9 mm, vias 0 -> 1
- net /MCU/TEMP_IRQ: track 0.00 -> 28.6 mm, vias 0 -> 3
- net /MCU/nRESET: track 0.00 -> 28.4 mm, vias 0 -> 2
- net +12V: track 65.9 -> 93.3 mm, vias 3 -> 4
- net VBUS: track 0.00 -> 26.1 mm, vias 0 -> 4
- net /MCU/RCC_OSC32_IN: track 0.00 -> 23.9 mm
- net /MCU/RXD: track 0.00 -> 23.1 mm, vias 0 -> 1
- net /MCU/USB_D+: track 0.00 -> 22.9 mm
- net /MCU/TXD: track 0.00 -> 22.4 mm, vias 0 -> 1
- net /LED driver/LED_G: track 3.41 -> 24.1 mm, vias 1 -> 2
- net /LED driver/LED_R: track 3.68 -> 24.1 mm, vias 1 -> 2
- net /MCU/USB_D-: track 0.00 -> 20.3 mm
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- added copper zone on B.Cu, net GND
- added copper zone on F.Cu, net Net-(C14-Pad1)
Other:
- net class Default: clearance 0.2032 -> 0.15; trace_width 0.2032 -> 0.15; via_dia 0.762 -> 0.6; via_drill 0.381 -> 0.35
- rule solder_mask_min_width: 0.25 -> 0.000051
- rule trace_clearance: 0.2032 -> 0.15
- rule trace_min: 0.1524 -> 0.015
- rule via_min_size: 0.508 -> 0.06

Commit message: layouting
Parts:
- added D5: BAT54S, Package_TO_SOT_SMD:SOT-23, F.Cu at (278.4, 176.2)
- added D6: BAT54S, Package_TO_SOT_SMD:SOT-23, F.Cu at (283.2, 173.3)
- added J6: Screw_Terminal_01x04, TerminalBlock_Phoenix:TerminalBlock_Phoenix_PT-1,5-4-3.5-H_1x04_P3.50mm_Horizontal, F.Cu at (261.6, 170.2)
- added R22: 10R, Resistor_SMD:R_0805_2012Metric_Pad1.15x1.40mm_HandSolder, F.Cu at (278.6, 169.5)
- added R23: 1K, Resistor_SMD:R_0805_2012Metric_Pad1.15x1.40mm_HandSolder, F.Cu at (266.6, 179.2)
- added R24: 10K, Resistor_SMD:R_0805_2012Metric_Pad1.15x1.40mm_HandSolder, F.Cu at (280.0, 151.1)
- added R25: 10R, Resistor_SMD:R_0805_2012Metric_Pad1.15x1.40mm_HandSolder, F.Cu at (271.3, 179.2)
- added R26: 1K, Resistor_SMD:R_0805_2012Metric_Pad1.15x1.40mm_HandSolder, F.Cu at (266.6, 182.1)
- added R27: 10K, Resistor_SMD:R_0805_2012Metric_Pad1.15x1.40mm_HandSolder, F.Cu at (283.3, 169.5)
- added U4: CCS811, Package_LGA:AMS_LGA-10-1EP_2.7x4mm_P0.6mm, F.Cu at (262.2, 180.4)
- added U7: BME280, Package_LGA:Bosch_LGA-8_2.5x2.5mm_P0.65mm_ClockwisePinNumbering, F.Cu at (275.7, 180.6)
- moved R5 163.6 mm to (179.1, 114.7), turned to 90 degrees
- moved D1 160.8 mm to (175.9, 111.4), turned to 270 degrees
- moved SW1 0.45 mm to (205.7, 105.4)
- moved C2 0.32 mm to (213.0, 113.3)
- moved R1 0.32 mm to (213.0, 111.4)
- moved IC1 0.32 mm to (223.5, 111.4)
- moved J1 0.32 mm to (208.3, 121.0)
- moved J2 0.32 mm to (201.9, 122.9)
Connections:
- IC2 pad 14: Net-(IC2-Pad14) -> /BLE/BLE_nRESET
- IC2 pad 15: Net-(IC2-Pad15) -> /BLE/BLE_IRQ
- IC2 pad 18: /BLE/BLE_IRQ -> /MCU/LED
Routing:
- net /BLE/BLE_nRESET: track 0.00 -> 11.2 mm
- net Net-(Q6-Pad1): track 0.00 -> 5.47 mm
- net Net-(Q6-Pad2): track 0.00 -> 3.85 mm
- net /BLE/BLE_nCS: track 11.2 -> 10.5 mm
- net /BLE/BLE_IRQ: track 13.7 -> 14.2 mm, vias 2 -> 0
- net GND: vias 66 -> 89

Commit message: dev
Parts:
- removed C14, C17: 1uF X5R, Capacitors_SMD:C_0805_HandSoldering
- removed C15, C18, C3, C4, C5, C8: 100nF, Capacitors_SMD:C_0805_HandSoldering
- removed C16: 10nF X7R, Capacitors_SMD:C_0805_HandSoldering
- removed C2: 1uF, Capacitors_SMD:C_0805_HandSoldering
- removed C6, C7: 4.3pF, Capacitors_SMD:C_0805_HandSoldering
- removed D3, D4: MBR0520, Diodes_SMD:D_SOD-123
- removed IC1: SPBTLE-RF0, RF_Modules:ST_SPBTLE
- removed IC2: STM32L052K8Tx, Housings_QFP:LQFP-32_7x7mm_Pitch0.8mm
- removed IC6: LD3985M33R_SOT23, TO_SOT_Packages_SMD:SOT-23-5_HandSoldering
- removed J1: Conn_ARM_JTAG_SWD_10, Pin_Headers:Pin_Header_Straight_2x05_Pitch1.27mm_SMD
- removed J2: COM, Pin_Headers:Pin_Header_Straight_1x06_Pitch2.54mm
- removed J5: USB_B_Micro, Connectors:USB_Micro-B
- removed Q6: BSS138, TO_SOT_Packages_SMD:SOT-23_Handsoldering
- removed R1: 47K, Resistors_SMD:R_0805_HandSoldering
- removed R14: 100K, Resistors_SMD:R_0805_HandSoldering
- removed R15: 1K5, Resistors_SMD:R_0805_HandSoldering
- removed R16, R3, R4: 10K, Resistors_SMD:R_0805_HandSoldering
- removed R17: 36K, Resistors_SMD:R_0805_HandSoldering
- removed R18: 100, Resistors_SMD:R_0805_HandSoldering
- removed R2: FBead, Resistors_SMD:R_0805_HandSoldering
- removed SW1: SW_Push, Button_Switch_SMD:SW_SPST_B3S-1100
- removed U3: USBLC6-2SC6, TO_SOT_Packages_SMD:SOT-23-6_Handsoldering
- removed U4: CCS811, Package_LGA:AMS_LGA-10-1EP_2.7x4mm_P0.6mm
- removed U7: BME280, Package_LGA:Bosch_LGA-8_2.5x2.5mm_P0.65mm_ClockwisePinNumbering
- removed Y1: 32.768kHz, Crystals:Crystal_SMD_HC49-SD_HandSoldering
- added C19: 100nF, Capacitor_SMD:C_0805_2012Metric_Pad1.15x1.40mm_HandSolder, F.Cu at (176.5, 139.7)
- added C20: 100nF, Capacitor_SMD:C_0805_2012Metric_Pad1.15x1.40mm_HandSolder, F.Cu at (181.3, 139.7)
- added U1: WeMos_D1_mini, Module:WEMOS_D1_mini_light, F.Cu at (236.3, 126.5)
- C1, C10, C11, C9: footprint Capacitors_SMD:C_0805_HandSoldering -> Capacitor_SMD:C_0805_2012Metric_Pad1.15x1.40mm_HandSolder
- R10, R11, R12, R13, R19, R20, R21, R5, R6, R7, R8, R9: footprint Resistors_SMD:R_0805_HandSoldering -> Resistor_SMD:R_0805_2012Metric_Pad1.15x1.40mm_HandSolder
Connections:
- D2 pad 1: Net-(C14-Pad1) -> +5V
Routing:
- net +3V3: track 77.3 -> 30.4 mm, vias 7 -> 3
- net VCOM: track 28.6 -> 0.00 mm, vias 1 -> 0
- net /MCU/nRESET: track 28.4 -> 0.00 mm, vias 2 -> 0
- net VBUS: track 26.1 -> 0.00 mm, vias 4 -> 0
- net /MCU/RCC_OSC32_IN: track 23.9 -> 0.00 mm
- net /MCU/RXD: track 23.0 -> 0.00 mm, vias 1 -> 0
- net /MCU/USB_D+: track 22.9 -> 0.00 mm
- net /MCU/TXD: track 22.3 -> 0.00 mm, vias 1 -> 0
- net /MCU/USB_D-: track 20.3 -> 0.00 mm
- net Net-(C14-Pad1): track 20.2 -> 0.00 mm
- net /MCU/RCC_OSC32_OUT: track 19.8 -> 0.00 mm
- net /BLE/BLE_IRQ: track 14.2 -> 0.00 mm
- net /MCU/SYS_SWDIO: track 13.6 -> 0.00 mm, vias 2 -> 0
- net +5V: track 0.00 -> 13.6 mm
- net /MCU/SYS_SWCLK: track 13.5 -> 0.00 mm, vias 2 -> 0
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- removed copper zone on F.Cu, net Net-(C14-Pad1)
