File: pcb/rgb_controller.kicad_pcb (KiCad board)
At the start: 2 copper layers, 50 x 75 mm, 75 parts, among them IC1 SPBTLE-RF0, IC2 STM32L052K8Tx, IC3 PM8834, IC4 PM8834, IC5 LD1117S50TR_SOT223, IC6 LD3985M33R_SOT23, J1 Conn_ARM_JTAG_SWD_10, J2 COM, J3 Screw_Terminal_01x02, J4 Screw_Terminal_01x06, J5 USB_B_Micro, J6 Screw_Terminal_01x04, Q1 IRF3205SPBF, Q2 IRF3205SPBF, Q3 IRF3205SPBF, Q4 IRF3205SPBF, Q6 BSS138, SW1 SW_Push, U2 LM75B, U3 USBLC6-2SC6, U4 CCS811, U5 TSL2550D, U7 BME280, Y1 32.768kHz

Commit message: ESP wroom module
Parts:
- removed the C5 at (234.0, 117.2)
- removed the C6 at (243.2, 125.1)
- removed the C7 at (243.2, 120.7)
- removed the D3 at (205.4, 139.4)
- removed the IC1 at (223.5, 111.4)
- removed the IC2 at (226.4, 120.7)
- removed the J1 at (208.3, 121.0)
- removed J5: USB_B_Micro, Connectors:USB_Micro-B
- removed Q6: BSS138, TO_SOT_Packages_SMD:SOT-23_Handsoldering
- removed the R1 at (213.0, 111.4)
- removed the R14 at (208.9, 133.0)
- removed the R15 at (210.8, 133.0)
- removed the R16 at (209.2, 125.7)
- removed the R17 at (216.5, 133.0)
- removed the R2 at (234.0, 119.1)
- removed R20: 4K7, Resistors_SMD:R_0805_HandSoldering
- removed the R3 at (230.2, 127.0)
- removed the U3 at (209.2, 128.6)
- removed U7: BME280, Package_LGA:Bosch_LGA-8_2.5x2.5mm_P0.65mm_ClockwisePinNumbering
- removed Y1: 32.768kHz, Crystals:Crystal_SMD_HC49-SD_HandSoldering
- added C17: 100nF, Capacitor_SMD:C_0805_2012Metric_Pad1.15x1.40mm_HandSolder, F.Cu at (294.6, 129.5)
- added C18: 15nF, Capacitor_SMD:C_0805_2012Metric_Pad1.15x1.40mm_HandSolder, F.Cu at (155.3, 158.7)
- added C4: 100nF, Capacitor_SMD:C_0805_2012Metric_Pad1.15x1.40mm_HandSolder, F.Cu at (218.0, 184.2)
- added D7: MMSZ5240BT1G, Diode_SMD:D_SOD-123, F.Cu at (156.2, 152.1)
- added Q5: IRF9540N, Package_TO_SOT_SMD:TO-263-2, F.Cu at (188.4, 153.9)
- added SW2: SW_Push, Button_Switch_SMD:SW_SPST_B3S-1000, F.Cu at (286.7, 132.3)
- added U1: ESP32-WROOM-32D, RF_Module:ESP32-WROOM-32, F.Cu at (225.4, 116.1)
- C1: renamed from C4; footprint Capacitors_SMD:C_0805_HandSoldering -> Capacitor_SMD:C_0805_2012Metric_Pad1.15x1.40mm_HandSolder
- C10: renamed from C13; footprint Capacitors_Tantalum_SMD:CP_Tantalum_Case-C_EIA-6032-28_Hand -> Capacitor_Tantalum_SMD:CP_EIA-6032-28_Kemet-C_Pad2.25x2.35mm_HandSolder
- C11: renamed from C14; footprint Capacitors_SMD:C_0805_HandSoldering -> Capacitor_SMD:C_0805_2012Metric_Pad1.15x1.40mm_HandSolder
- C12: renamed from C15; footprint Capacitors_SMD:C_0805_HandSoldering -> Capacitor_SMD:C_0805_2012Metric_Pad1.15x1.40mm_HandSolder
- C13: renamed from C16; footprint Capacitors_SMD:C_0805_HandSoldering -> Capacitor_SMD:C_0805_2012Metric_Pad1.15x1.40mm_HandSolder
- C14: renamed from C17; footprint Capacitors_SMD:C_0805_HandSoldering -> Capacitor_SMD:C_0805_2012Metric_Pad1.15x1.40mm_HandSolder
- C15: renamed from C18; footprint Capacitors_SMD:C_0805_HandSoldering -> Capacitor_SMD:C_0805_2012Metric_Pad1.15x1.40mm_HandSolder
- C16: renamed from C1; footprint Capacitors_SMD:C_0805_HandSoldering -> Capacitor_SMD:C_0805_2012Metric_Pad1.15x1.40mm_HandSolder
- C2: value 1uF -> 10uF; footprint Capacitors_SMD:C_0805_HandSoldering -> Capacitor_Tantalum_SMD:CP_EIA-6032-28_Kemet-C_Pad2.25x2.35mm_HandSolder
- C3: footprint Capacitors_SMD:C_0805_HandSoldering -> Capacitor_SMD:C_0805_2012Metric_Pad1.15x1.40mm_HandSolder
- C5: renamed from C8; footprint Capacitors_SMD:C_0805_HandSoldering -> Capacitor_SMD:C_0805_2012Metric_Pad1.15x1.40mm_HandSolder
- C6: renamed from C9; footprint Capacitors_SMD:C_0805_HandSoldering -> Capacitor_SMD:C_0805_2012Metric_Pad1.15x1.40mm_HandSolder
- C7: renamed from C10; footprint Capacitors_SMD:C_0805_HandSoldering -> Capacitor_SMD:C_0805_2012Metric_Pad1.15x1.40mm_HandSolder
- C8: renamed from C11; footprint Capacitors_SMD:C_0805_HandSoldering -> Capacitor_SMD:C_0805_2012Metric_Pad1.15x1.40mm_HandSolder
- C9: renamed from C12; footprint Capacitors_Tantalum_SMD:CP_Tantalum_Case-C_EIA-6032-28_Hand -> Capacitor_Tantalum_SMD:CP_EIA-6032-28_Kemet-C_Pad2.25x2.35mm_HandSolder
- R10: renamed from R6; footprint Resistors_SMD:R_0805_HandSoldering -> Resistor_SMD:R_0805_2012Metric_Pad1.15x1.40mm_HandSolder
- R11: renamed from R7; footprint Resistors_SMD:R_0805_HandSoldering -> Resistor_SMD:R_0805_2012Metric_Pad1.15x1.40mm_HandSolder
- R12: renamed from R8; footprint Resistors_SMD:R_0805_HandSoldering -> Resistor_SMD:R_0805_2012Metric_Pad1.15x1.40mm_HandSolder
- R13: renamed from R9; footprint Resistors_SMD:R_0805_HandSoldering -> Resistor_SMD:R_0805_2012Metric_Pad1.15x1.40mm_HandSolder
- R14: renamed from R10; footprint Resistors_SMD:R_0805_HandSoldering -> Resistor_SMD:R_0805_2012Metric_Pad1.15x1.40mm_HandSolder
- R15: renamed from R12; footprint Resistors_SMD:R_0805_HandSoldering -> Resistor_SMD:R_0805_2012Metric_Pad1.15x1.40mm_HandSolder
- R16: renamed from R11; footprint Resistors_SMD:R_0805_HandSoldering -> Resistor_SMD:R_0805_2012Metric_Pad1.15x1.40mm_HandSolder
- R17: renamed from R13; footprint Resistors_SMD:R_0805_HandSoldering -> Resistor_SMD:R_0805_2012Metric_Pad1.15x1.40mm_HandSolder
- R18: value 100 -> 10K; footprint Resistors_SMD:R_0805_HandSoldering -> Resistor_SMD:R_0805_2012Metric_Pad1.15x1.40mm_HandSolder
- R19: value 4K7 -> 10K; footprint Resistors_SMD:R_0805_HandSoldering -> Resistor_SMD:R_0805_2012Metric_Pad1.15x1.40mm_HandSolder
- R7: renamed from R4; footprint Resistors_SMD:R_0805_HandSoldering -> Resistor_SMD:R_0805_2012Metric_Pad1.15x1.40mm_HandSolder
- R8: renamed from R5; footprint Resistors_SMD:R_0805_HandSoldering -> Resistor_SMD:R_0805_2012Metric_Pad1.15x1.40mm_HandSolder
- R9: renamed from R21; footprint Resistors_SMD:R_0805_HandSoldering -> Resistor_SMD:R_0805_2012Metric_Pad1.15x1.40mm_HandSolder
- SW1: footprint Button_Switch_SMD:SW_SPST_B3S-1100 -> Button_Switch_SMD:SW_SPST_B3S-1000
- U4: value CCS811 -> Si7021-A20; footprint Package_LGA:AMS_LGA-10-1EP_2.7x4mm_P0.6mm -> Package_DFN_QFN:DFN-6-1EP_3x3mm_P1mm_EP1.5x2.4mm
- moved R18 76.1 mm to (294.6, 132.5), turned to 0 degrees
- moved C3 67.9 mm to (213.3, 184.2), turned to 0 degrees
- moved R19 56.8 mm to (202.4, 87.4), turned to 0 degrees
- moved C2 49.6 mm to (262.6, 115.8), turned to 0 degrees
- moved J2 44.9 mm to (246.7, 120.1)
- moved R7 43.5 mm to (256.9, 126.5)
- moved C1 29.9 mm to (263.9, 125.4)
- moved C5 29.6 mm to (263.6, 121.5)
- moved U4 28.4 mm to (262.0, 152.0)
- moved SW1 1.08 mm to (205.7, 104.3)
- renumbered D5 to D1, D6 to D2, D1 to D3, D2 to D6, IC3 to IC1, IC4 to IC2, IC5 to IC3, IC6 to IC4, J6 to J1, J4 to J3, J3 to J4, R22 to R1, R23 to R2, R24 to R3, R25 to R4, R26 to R5, R27 to R6, U5 to U3
Connections:
- net /MCU/TEMP_IRQ renamed Net-(R9-Pad2)
- net /MCU/nRESET renamed /MCU/EN
- C3 pad 1: +3V3 -> Net-(C3-Pad1)
- J2 pad 4: /MCU/TXD -> /MCU/RXD0
- J4 pad 1: +12V -> Net-(J4-Pad1)
- R18 pad 1: /MCU/USB_RENUMn -> +3V3
- R18 pad 2: Net-(Q6-Pad1) -> /MCU/IO0
- R19 pad 1: /MCU/I2C1_SCL -> Net-(C18-Pad1)
- R19 pad 2: +3V3 -> GND
- R2 pad 1: Net-(C19-Pad1) -> Net-(C3-Pad1)
- R3 pad 1: Net-(C19-Pad1) -> Net-(C3-Pad1)
- R8 pad 1: /MCU/LED -> /MCU/IO13
Routing:
- net +3V3: track 77.3 -> 36.2 mm, vias 7 -> 3
- net VCOM: track 28.6 -> 0.00 mm, vias 1 -> 0
- net /MCU/EN: track 28.4 -> 0.23 mm, vias 2 -> 0
- net VBUS: track 26.1 -> 0.00 mm, vias 4 -> 0
- net /MCU/RCC_OSC32_IN: track 23.9 -> 0.00 mm
- net /MCU/RXD: track 23.0 -> 0.00 mm, vias 1 -> 0
- net /MCU/USB_D+: track 22.9 -> 0.00 mm
- net /MCU/TXD: track 22.3 -> 0.00 mm, vias 1 -> 0
- net /MCU/USB_D-: track 20.3 -> 0.00 mm
- net /MCU/RCC_OSC32_OUT: track 19.8 -> 0.00 mm
- net /BLE/BLE_IRQ: track 14.2 -> 0.00 mm
- net /MCU/SYS_SWDIO: track 13.6 -> 0.00 mm, vias 2 -> 0
- net /MCU/SYS_SWCLK: track 13.5 -> 0.00 mm, vias 2 -> 0
- net /LED driver/LED_W: track 23.2 -> 11.6 mm, vias 2 -> 1
- net /LED driver/LED_B: track 22.5 -> 11.0 mm, vias 2 -> 1
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
Commit message: backup
Parts:
- added C19: 100nF, Capacitor_SMD:C_0805_2012Metric_Pad1.15x1.40mm_HandSolder, F.Cu at (119.7, 211.1)
- added C20: 100nF, Capacitor_SMD:C_0805_2012Metric_Pad1.15x1.40mm_HandSolder, F.Cu at (125.0, 206.5)
- added H1: MountingHole, MountingHole:MountingHole_3.2mm_M3, F.Cu at (205.0, 155.0)
- added H2: MountingHole, MountingHole:MountingHole_3.2mm_M3, F.Cu at (155.0, 155.0)
- added H3: MountingHole, MountingHole:MountingHole_3.2mm_M3, F.Cu at (155.0, 245.0)
- added H4: MountingHole, MountingHole:MountingHole_3.2mm_M3, F.Cu at (205.0, 245.0)
- added U5: Si7021-A20, Package_DFN_QFN:DFN-6-1EP_3x3mm_P1mm_EP1.5x2.4mm, F.Cu at (120.0, 207.3)
- D4, D6: footprint Diodes_SMD:D_SOD-123 -> Diode_SMD:D_SOD-123
- U4: value Si7021-A20 -> BMP280; footprint Package_DFN_QFN:DFN-6-1EP_3x3mm_P1mm_EP1.5x2.4mm -> Package_LGA:Bosch_LGA-8_2x2.5mm_P0.65mm_ClockwisePinNumbering
- moved U4 149.0 mm to (124.7, 209.8)
- moved C17 137.2 mm to (157.6, 138.7)
- moved R18 137.2 mm to (157.4, 135.2)
- moved R19 136.5 mm to (160.0, 217.2), turned to 90 degrees
- moved SW2 128.1 mm to (158.6, 128.1)
- moved D1 112.8 mm to (379.0, 125.2)
- moved D2 112.8 mm to (383.8, 122.2)
- moved J1 112.8 mm to (362.2, 119.1)
- moved R1 112.8 mm to (379.2, 118.5)
- moved R2 112.8 mm to (367.2, 128.1)
- moved R3 112.8 mm to (380.6, 100.1)
- moved R4 112.8 mm to (371.9, 128.1)
- moved R5 112.8 mm to (367.2, 131.1)
- moved R6 112.8 mm to (383.9, 118.5)
- moved C3 112.8 mm to (313.9, 133.1)
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Connections:
- net Net-(C3-Pad1) renamed /MCU/IN1
- net Net-(C4-Pad1) renamed /MCU/IN2
- U4 pad 1: Net-(U4-Pad1) -> GND
- U4 pad 2: Net-(U4-Pad2) -> +3V3
- U4 pad 3: Net-(U4-Pad3) -> /MCU/I2C1_SDA
- U4 pad 4: Net-(U4-Pad4) -> /MCU/I2C1_SCL
- U4 pad 5: Net-(U4-Pad5) -> GND
- U4 pad 6: Net-(U4-Pad6) -> +3V3
- U4 pad 7: Net-(U4-Pad7) -> GND
Routing:
- net +12V: track 93.3 -> 32.2 mm
- net +3V3: track 36.2 -> 4.49 mm, vias 3 -> 0
- net /MCU/I2C1_SDA: track 30.2 -> 0.00 mm, vias 4 -> 0
- net /MCU/I2C1_SCL: track 28.5 -> 0.00 mm, vias 4 -> 0
- net Net-(R9-Pad2): track 25.1 -> 0.00 mm, vias 3 -> 0
- net Net-(C10-Pad1): track 19.3 -> 0.00 mm
- net Net-(IC1-Pad7): track 19.3 -> 0.00 mm
- net Net-(C11-Pad1): track 20.2 -> 5.35 mm
- net Net-(IC2-Pad5): track 14.3 -> 0.00 mm
- net /LED driver/LED_R: track 14.2 -> 2.25 mm, vias 1 -> 0
- net /LED driver/LED_G: track 13.4 -> 1.99 mm, vias 1 -> 0
- net Net-(IC1-Pad5): track 10.8 -> 0.00 mm
- net /LED driver/DRIVER_W: track 31.4 -> 21.4 mm
- net /LED driver/LED_W: track 11.6 -> 1.99 mm, vias 1 -> 0
- net /LED driver/LED_B: track 11.0 -> 2.25 mm, vias 1 -> 0
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- removed copper zone on F.Cu, net Net-(C11-Pad1)
Other:
- board size 50 x 75 mm -> 60 x 100 mm
