File: pcb/rgb_controller.sch (KiCad schematic (older format))
At the start: 3 parts, among them U1 M95256-WMN6P

Commit message: WIP
Parts:
- removed BT1: CR2032, Connectors:CR2032H, symbol Device:Battery_Cell
- removed C1: 1uF X5R, Capacitors_SMD:C_0805_HandSoldering, symbol Device:C
- removed U1: M95256-WMN6P, Housings_SOIC:SOIC-8_3.9x4.9mm_Pitch1.27mm, symbol Memory_EEPROM:M95256-WMN6P
Connections:
- net labels removed: +BATT, GND
- wire segments 17 -> 22
Changed lines of the file:
@@
 EESchema Schematic File Version 4
+LIBS:rgb_controller-cache
 EELAYER 26 0
 EELAYER END
 $Descr A4 11693 8268
 encoding utf-8
-Sheet 1 4
+Sheet 1 7
 Title "Overview"
-Date "2019-02-22"
+Date "2019-02-23"
 Rev ""
 Comp "HuizePD"
@@
 F7 "BLE_IRQ" O L 6700 3250 50
 $EndSheet
-$Comp
-L Memory_EEPROM:M95256-WMN6P U1
-U 1 1 5C6FBCA8
-P 10100 5750
-F 0 "U1" H 10100 6228 50  0000 C CNN
-F 1 "M95256-WMN6P" H 10100 6137 50  0000 C CNN
-F 2 "Housings_SOIC:SOIC-8_3.9x4.9mm_Pitch1.27mm" H 10100 5750 50  0001 C CNN
-F 3 "http://www.st.com/content/ccc/resource/technical/document/datasheet/9d/75/f0/3e/76/00/4c/0b/CD00103810.pdf/files/CD00103810.pdf/jcr:content/translations/en.CD00103810.pdf" H 10100 5750 50  0001 C CNN
-	1    10100 5750
-	1    0    0    -1
-$EndComp
 $Comp
 L power:+3V3 #PWR06
@@
 Wire Wire Line
 	5100 5750 5100 5700
-$Comp
-L power:+BATT #PWR03
-U 1 1 5C717483
-P 1700 2200
-F 0 "#PWR03" H 1700 2050 50  0001 C CNN
-F 1 "+BATT" H 1715 2373 50  0000 C CNN
-F 2 "" H 1700 2200 50  0001 C CNN
-F 3 "" H 1700 2200 50  0001 C CNN
-	1    1700 2200
-	1    0    0    -1
-$EndComp
-Wire Wire Line
-	1700 2200 1700 2950
-$Comp
-L Device:C C1
-U 1 1 5C72005E
-P 1300 2400
-F 0 "C1" H 1415 2446 50  0000 L CNN
-F 1 "1uF X5R" H 1415 2355 50  0000 L CNN
-F 2 "Capacitors_SMD:C_0805_HandSoldering" H 1338 2250 50  0001 C CNN
-F 3 "~" H 1300 2400 50  0001 C CNN
-	1    1300 2400
-	1    0    0    -1
-$EndComp
-$Comp
-L power:+BATT #PWR01
-U 1 1 5C72017F
-P 1300 2200
-F 0 "#PWR01" H 1300 2050 50  0001 C CNN
-F 1 "+BATT" H 1315 2373 50  0000 C CNN
-F 2 "" H 1300 2200 50  0001 C CNN
-F 3 "" H 1300 2200 50  0001 C CNN
-	1    1300 2200
-	1    0    0    -1
-$EndComp
-Wire Wire Line
-	1300 2250 1300 2200
-Wire Wire Line
-	1300 2550 1300 2600
-$Comp
-L power:GND #PWR02
-U 1 1 5C72335C
-P 1300 2600
-F 0 "#PWR02" H 1300 2350 50  0001 C CNN
-F 1 "GND" H 1305 2427 50  0000 C CNN
-F 2 "" H 1300 2600 50  0001 C CNN
-F 3 "" H 1300 2600 50  0001 C CNN
-	1    1300 2600
-	1    0    0    -1
-$EndComp
-$Comp
-L Device:Battery_Cell BT1
-U 1 1 5C72C35B
-P 2150 2500
-F 0 "BT1" H 2268 2596 50  0000 L CNN
-F 1 "CR2032" H 2268 2505 50  0000 L CNN
-F 2 "Connectors:CR2032H" V 2150 2560 50  0001 C CNN
-F 3 "~" V 2150 2560 50  0001 C CNN
-	1    2150 2500
-	1    0    0    -1
-$EndComp
-$Comp
-L power:GND #PWR05
-U 1 1 5C72C4E5
-P 2150 2650
-F 0 "#PWR05" H 2150 2400 50  0001 C CNN
-F 1 "GND" H 2155 2477 50  0000 C CNN
-F 2 "" H 2150 2650 50  0001 C CNN
-F 3 "" H 2150 2650 50  0001 C CNN
-	1    2150 2650
-	1    0    0    -1
-$EndComp
-Wire Wire Line
-	2150 2650 2150 2600
-$Comp
-L power:+BATT #PWR04
-U 1 1 5C72E1A5
-P 2150 2200
-F 0 "#PWR04" H 2150 2050 50  0001 C CNN
-F 1 "+BATT" H 2165 2373 50  0000 C CNN
-F 2 "" H 2150 2200 50  0001 C CNN
-F 3 "" H 2150 2200 50  0001 C CNN
-	1    2150 2200
-	1    0    0    -1
-$EndComp
-Wire Wire Line
-	2150 2200 2150 2300
 $Sheet
 S 4850 2500 1450 1800
@@
 F9 "I2C1_SCL" B R 6300 3900 50
 F10 "I2C1_SDA" B R 6300 4000 50
+F11 "LED_R" O L 4850 3850 50
+F12 "LED_G" O L 4850 3950 50
+F13 "LED_B" O L 4850 4050 50
+F14 "LED_W" O L 4850 4150 50
 $EndSheet
 Wire Wire Line
@@
 F0 "Temperature" 50
 F1 "rgb_controller-temp.sch" 50
-F2 "TEMP_SDA" B L 6700 3900 50
-F3 "TEMP_SCL" B L 6700 4000 50
+F2 "TEMP_SDA" B L 6700 4000 50
+F3 "TEMP_SCL" B L 6700 3900 50
 F4 "TEMP_IRQ" O L 6700 4150 50
 $EndSheet
 Wire Wire Line
-	6300 4000 6700 4000
-Wire Wire Line
-	6700 3900 6300 3900
+	6300 4000 6550 4000
 Wire Wire Line
 	6300 4150 6700 4150
+$Sheet
+S 3850 3750 700  500
+U 5C726A30
+F0 "LED driver" 50
+F1 "rgb_controller-led-driver.sch" 50
+F2 "LED_R" I R 4550 3850 50
+F3 "LED_G" I R 4550 3950 50
+F4 "LED_B" I R 4550 4050 50
+F5 "LED_W" I R 4550 4150 50
+$EndSheet
+Wire Wire Line
+	4550 4150 4850 4150
+Wire Wire Line
+	4850 4050 4550 4050
+Wire Wire Line
+	4550 3950 4850 3950
+Wire Wire Line
+	4850 3850 4550 3850
+$Sheet
+S 3050 850  1850 850
+U 5C739DCD
+F0 "Power supply" 50
+F1 "led_driver-power.sch" 50
+$EndSheet
+$Sheet
+S 6700 4550 700  500
+U 5C7F522E
+F0 "Light Sensor" 50
+F1 "led_driver-light_sensor.sch" 50
+F2 "I2C_SCL" B L 6700 4750 50
+F3 "I2C_SDA" B L 6700 4850 50
+$EndSheet
+Wire Wire Line
+	6700 4750 6600 4750
+Wire Wire Line
+	6700 3900 6600 3900
+Wire Wire Line
+	6600 4750 6600 3900
+Connection ~ 6600 3900
+Wire Wire Line
+	6600 3900 6300 3900
+Wire Wire Line
+	6550 4000 6550 4850
+Wire Wire Line
+	6550 4850 6700 4850
+Connection ~ 6550 4000
+Wire Wire Line
+	6550 4000 6700 4000
 $EndSCHEMATC

Commit message: dev
Changed lines of the file:
@@
 EESchema Schematic File Version 4
 LIBS:rgb_controller-cache
-EELAYER 29 0
+EELAYER 30 0
 EELAYER END
 $Descr A4 11693 8268
 encoding utf-8
-Sheet 1 7
+Sheet 1 6
 Title "Overview"
 Date "2019-02-23"
@@
 Comment4 "Author: Sander Huisman"
 $EndDescr
-$Sheet
-S 6700 2500 700  1050
-U 5C6DADA9
-F0 "BLE" 50
-F1 "rgb_controller-ble.sch" 50
-F2 "BLE_nRESET" I L 6700 3350 50
-F3 "BLE_nCS" I L 6700 3150 50
-F4 "SPI_MOSI" I L 6700 2850 50
-F5 "SPI_MISO" O L 6700 2950 50
-F6 "SPI_CLK" I L 6700 2750 50
-F7 "BLE_IRQ" O L 6700 3250 50
-$EndSheet
 $Comp
 L power:+3V3 #PWR06
@@
 F14 "LED_W" O L 4850 4150 50
 $EndSheet
-Wire Wire Line
-	6300 2950 6700 2950
-Wire Wire Line
-	6700 2850 6300 2850
-Wire Wire Line
-	6700 2750 6300 2750
-Wire Wire Line
-	6700 3150 6300 3150
-Wire Wire Line
-	6700 3250 6300 3250
-Wire Wire Line
-	6700 3350 6300 3350
 $Sheet
 S 6700 3750 700  550
