File: pcb/rgb_controller.sch (KiCad schematic (older format))
At the start: 0 parts

Commit message: ESP wroom module
Changed lines of the file:
@@
 EESchema Schematic File Version 4
 LIBS:rgb_controller-cache
-EELAYER 29 0
+EELAYER 30 0
 EELAYER END
 $Descr A4 11693 8268
 encoding utf-8
-Sheet 1 7
+Sheet 1 6
 Title "Overview"
 Date "2019-02-23"
@@
 Comment4 "Author: Sander Huisman"
 $EndDescr
-$Sheet
-S 6700 2500 700  1050
-U 5C6DADA9
-F0 "BLE" 50
-F1 "rgb_controller-ble.sch" 50
-F2 "BLE_nRESET" I L 6700 3350 50
-F3 "BLE_nCS" I L 6700 3150 50
-F4 "SPI_MOSI" I L 6700 2850 50
-F5 "SPI_MISO" O L 6700 2950 50
-F6 "SPI_CLK" I L 6700 2750 50
-F7 "BLE_IRQ" O L 6700 3250 50
-$EndSheet
 $Comp
-L power:+3V3 #PWR06
+L power:+3V3 #PWR01
 U 1 1 5C71583F
 P 5100 5700
-F 0 "#PWR06" H 5100 5550 50  0001 C CNN
+F 0 "#PWR01" H 5100 5550 50  0001 C CNN
 F 1 "+3V3" H 5115 5873 50  0000 C CNN
 F 2 "" H 5100 5700 50  0001 C CNN
@@
 $EndComp
 $Comp
-L power:VDD #PWR07
+L power:VDD #PWR02
 U 1 1 5C7158D4
 P 5300 5700
-F 0 "#PWR07" H 5300 5550 50  0001 C CNN
+F 0 "#PWR02" H 5300 5550 50  0001 C CNN
 F 1 "VDD" H 5317 5873 50  0000 C CNN
 F 2 "" H 5300 5700 50  0001 C CNN
@@
 F0 "MCU" 50
 F1 "rgb_controller-mcu.sch" 50
-F2 "SPI1_CLK" O R 6300 2750 50
-F3 "SPI1_MISO" I R 6300 2950 50
-F4 "SPI1_MOSI" O R 6300 2850 50
-F5 "BLE_nCS" O R 6300 3150 50
-F6 "BLE_IRQ" O R 6300 3250 50
-F7 "BLE_nRESET" O R 6300 3350 50
-F8 "TEMP_IRQ" I R 6300 4150 50
-F9 "I2C1_SCL" B R 6300 3900 50
-F10 "I2C1_SDA" B R 6300 4000 50
-F11 "LED_R" O L 4850 3850 50
-F12 "LED_G" O L 4850 3950 50
-F13 "LED_B" O L 4850 4050 50
-F14 "LED_W" O L 4850 4150 50
+F2 "I2C1_SCL" B R 6300 3900 50
+F3 "I2C1_SDA" B R 6300 4000 50
+F4 "LED_R" O L 4850 3850 50
+F5 "LED_G" O L 4850 3950 50
+F6 "LED_B" O L 4850 4050 50
+F7 "LED_W" O L 4850 4150 50
 $EndSheet
-Wire Wire Line
-	6300 2950 6700 2950
-Wire Wire Line
-	6700 2850 6300 2850
-Wire Wire Line
-	6700 2750 6300 2750
-Wire Wire Line
-	6700 3150 6300 3150
-Wire Wire Line
-	6700 3250 6300 3250
-Wire Wire Line
-	6700 3350 6300 3350
 $Sheet
 S 6700 3750 700  550
@@
 F2 "TEMP_SDA" B L 6700 4000 50
 F3 "TEMP_SCL" B L 6700 3900 50
-F4 "TEMP_IRQ" O L 6700 4150 50
 $EndSheet
 Wire Wire Line
 	6300 4000 6550 4000
-Wire Wire Line
-	6300 4150 6700 4150
 $Sheet
 S 3850 3750 700  500

Commit message: backup
Parts:
- added H1, H2, H3, H4: MountingHole, MountingHole:MountingHole_3.2mm_M3, symbol Mechanical:MountingHole
Changed lines of the file:
@@
 Wire Wire Line
 	6550 4000 6700 4000
+$Comp
+L Mechanical:MountingHole H1
+U 1 1 5DA6DF2D
+P 3450 6500
+F 0 "H1" H 3550 6546 50  0000 L CNN
+F 1 "MountingHole" H 3550 6455 50  0000 L CNN
+F 2 "MountingHole:MountingHole_3.2mm_M3" H 3450 6500 50  0001 C CNN
+F 3 "~" H 3450 6500 50  0001 C CNN
+	1    3450 6500
+	1    0    0    -1
+$EndComp
+$Comp
+L Mechanical:MountingHole H2
+U 1 1 5DA6E377
+P 3450 6700
+F 0 "H2" H 3550 6746 50  0000 L CNN
+F 1 "MountingHole" H 3550 6655 50  0000 L CNN
+F 2 "MountingHole:MountingHole_3.2mm_M3" H 3450 6700 50  0001 C CNN
+F 3 "~" H 3450 6700 50  0001 C CNN
+	1    3450 6700
+	1    0    0    -1
+$EndComp
+$Comp
+L Mechanical:MountingHole H3
+U 1 1 5DA6EAF1
+P 4150 6500
+F 0 "H3" H 4250 6546 50  0000 L CNN
+F 1 "MountingHole" H 4250 6455 50  0000 L CNN
+F 2 "MountingHole:MountingHole_3.2mm_M3" H 4150 6500 50  0001 C CNN
+F 3 "~" H 4150 6500 50  0001 C CNN
+	1    4150 6500
+	1    0    0    -1
+$EndComp
+$Comp
+L Mechanical:MountingHole H4
+U 1 1 5DA6EE69
+P 4150 6700
+F 0 "H4" H 4250 6746 50  0000 L CNN
+F 1 "MountingHole" H 4250 6655 50  0000 L CNN
+F 2 "MountingHole:MountingHole_3.2mm_M3" H 4150 6700 50  0001 C CNN
+F 3 "~" H 4150 6700 50  0001 C CNN
+	1    4150 6700
+	1    0    0    -1
+$EndComp
 $EndSCHEMATC
